File: 5806213/5806213.kicad_sch (KiCad schematic)
At the start: 242 parts

Commit message: Remove extranious labels
Connections:
- net AND Extend: no longer D?.2 (A), D?.2 (A), D?.2 (A), D?.2 (A), D?.2 (A), D?.2 (A), D?.2 (A), D?.2 (A), D?.2 (A), D?.2 (A), D?.2 (A), D?.2 (A), D?.2 (A), D?.2 (A), D?.2 (A), D?.2 (A), D?.2 (A), D?.2 (A), D?.2 (A), D?.2 (A), R?.2, R?.2, R?.2, R?.2, R?.2
- removed net OR Extend: D?.1 (K), D?.1 (K), D?.1 (K), D?.2 (A), D?.2 (A), D?.2 (A), D?.2 (A), D?.2 (A), D?.2 (A)
- new net: D?.1 (K), D?.2 (A), D?.2 (A) (x3)
- new net: D?.2 (A), D?.2 (A), D?.2 (A), D?.2 (A), R?.2 (x5)
Changed lines of the file:
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@@
-    (effects (font (size 1.27 1.27)) (justify left bottom))
-  )
-  (label "AND Extend" (at 135.89 218.44 0)
     (effects (font (size 1.27 1.27)) (justify left bottom))
   )
@@
     (effects (font (size 1.27 1.27)) (justify left bottom))
   )
-  (label "AND Extend" (at 135.89 356.87 0)
-    (effects (font (size 1.27 1.27)) (justify left bottom))
-  )
   (label "J07" (at 85.09 133.35 270)
     (effects (font (size 1.27 1.27)) (justify right bottom))
@@
     (effects (font (size 1.27 1.27)) (justify left bottom))
   )
-  (label "OR Extend" (at 137.16 499.11 0)
-    (effects (font (size 1.27 1.27)) (justify left bottom))
-  )
   (label "J05" (at 299.72 788.67 270)
     (effects (font (size 1.27 1.27)) (justify right bottom))
@@
     (effects (font (size 1.27 1.27)) (justify left bottom))
   )
-  (label "AND Extend" (at 417.83 355.6 0)
-    (effects (font (size 1.27 1.27)) (justify left bottom))
-  )
   (label "J11" (at 129.54 314.96 180)
     (effects (font (size 1.27 1.27)) (justify right bottom))
@@
     (effects (font (size 1.27 1.27)) (justify left bottom))
   )
-  (label "AND Extend" (at 585.47 218.44 0)
-    (effects (font (size 1.27 1.27)) (justify left bottom))
-  )
   (label "B08" (at 741.68 788.67 270)
     (effects (font (size 1.27 1.27)) (justify right bottom))
@@
     (effects (font (size 1.27 1.27)) (justify right bottom))
   )
-  (label "AND Extend" (at 416.56 218.44 0)
-    (effects (font (size 1.27 1.27)) (justify left bottom))
-  )
   (label "D02" (at 134.62 133.35 270)
     (effects (font (size 1.27 1.27)) (justify right bottom))
@@
     (effects (font (size 1.27 1.27)) (justify left bottom))
   )
-  (label "OR Extend" (at 412.75 499.11 0)
-    (effects (font (size 1.27 1.27)) (justify left bottom))
-  )
   (label "D09" (at 116.84 133.35 270)
     (effects (font (size 1.27 1.27)) (justify right bottom))
@@
     (effects (font (size 1.27 1.27)) (justify right bottom))
   )
-  (label "OR Extend" (at 730.25 505.46 0)
-    (effects (font (size 1.27 1.27)) (justify left bottom))
-  )
   (symbol (lib_id "Device:R_Small_US") (at 468.63 481.33 0) (unit 1)

Commit message: Remove extra labels
Connections:
- removed net AND Extend: D?.2 (A), D?.2 (A), D?.2 (A), D?.2 (A), D?.2 (A), D?.2 (A), D?.2 (A), D?.2 (A), D?.2 (A), D?.2 (A), D?.2 (A), D?.2 (A), R?.2, R?.2, R?.2
- new net: D?.2 (A), D?.2 (A), D?.2 (A), D?.2 (A), R?.2 (x3)
Changed lines of the file:
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@@
     (effects (font (size 1.27 1.27)) (justify right bottom))
-  )
-  (label "AND Extend" (at 137.16 443.23 0)
-    (effects (font (size 1.27 1.27)) (justify left bottom))
   )
   (label "+3V" (at 177.8 560.07 90)
@@
     (effects (font (size 1.27 1.27)) (justify right bottom))
   )
-  (label "AND Extend" (at 730.25 449.58 0)
-    (effects (font (size 1.27 1.27)) (justify left bottom))
-  )
   (label "+3V" (at 655.32 154.94 90)
     (effects (font (size 1.27 1.27)) (justify left bottom))
@@
     (effects (font (size 1.27 1.27)) (justify left bottom))
   )
-  (label "AND Extend" (at 412.75 443.23 0)
-    (effects (font (size 1.27 1.27)) (justify left bottom))
-  )
