File: 1130_backplane/01B-A1.kicad_sch (KiCad schematic)
At the start: 86 parts

Commit message: DN101-DN111 added to backplane schematics, DN111 01B-A1 connections made, 01B-B1 connections to be made when all signals on connectors
Connections:
- net +3V: no longer J271.b2 (Pin_b2), J340.b2 (Pin_b2)
- net +6V: no longer J340.a10 (Pin_a10), J341.a10 (Pin_a10)
- net -3V: no longer J340.a5 (Pin_a5), J341.a5 (Pin_a5)
- net +T_3: now reaches J277.a11 (Pin_a11)
- net -ARITH_CTRL_B: now reaches J277.a12 (Pin_a12)
- net -MULTIPLY_OP: now reaches J277.a2 (Pin_a2)
- net -OP_BIT_1: now reaches J277.a3 (Pin_a3)
- net -OP_BIT_1: now also J272.b12 (Pin_b12)
- net +OP_BIT_4: now reaches J277.a4 (Pin_a4)
- net +OP_BIT_4: now also J272.b11 (Pin_b11)
- net +OP_BIT_2: now reaches J277.a6 (Pin_a6)
- net +OP_BIT_2: now also J271.b6 (Pin_b6)
- net -DIVIDE_OP: now reaches J277.a7 (Pin_a7)
- net +OP_BIT_1: now reaches J277.a8 (Pin_a8)
- net +OP_BIT_1: now also J271.a6 (Pin_a6)
- net -DBL_WORD_ADDRESSING: now reaches J277.a9 (Pin_a9)
- net -OP_1011X: now reaches J277.b1 (Pin_b1)
- net -T_0: now reaches J277.b10 (Pin_b10)
- net +MULTIPLY_OP: now reaches J277.b11 (Pin_b11)
- net +OP_BIT_0: now reaches J277.b3 (Pin_b3)
- net -ADD_SUB_GATE_E: now reaches J277.b4 (Pin_b4)
- net +OP_BIT_3: now reaches J277.b5 (Pin_b5)
- net +OP_BIT_3: now also J272.b9 (Pin_b9)
- net -OP_BIT_3: now reaches J277.b6 (Pin_b6)
- net -OP_BIT_4: now reaches J277.b8 (Pin_b8)
- net -OP_BIT_4: now also J272.a9 (Pin_a9)
- net +E_CYCLES: now reaches J277.b9 (Pin_b9)
- net +E_CYCLES: now also J272.b5 (Pin_b5)
- net -ADD_SUB_OR_EOR_GATE: now reaches J341.a9 (Pin_a9)
- net -ADD_SUB_OR_EOR_GATE: now also J278.a8 (Pin_a8)
- net -ADD_SUB_EOR_GATE: now reaches J341.b9 (Pin_b9)
- net -ADD_SUB_EOR_GATE: now also J278.b8 (Pin_b8)
- net -MULTIPLY_E: now reaches J278.a1 (Pin_a1)
- net -XIO_E: now reaches J278.a11 (Pin_a11)
- net -I2_CYCLE: now reaches J278.a12 (Pin_a12)
- net -STORE_E: now reaches J278.a2 (Pin_a2)
- net -OP_BIT_2: now reaches J278.a3 (Pin_a3)
- net -OP_BIT_2: now also J272.b8 (Pin_b8)
- net +XIO_OP: now reaches J278.a4 (Pin_a4)
- net +XIO_OP: now also J271.a11 (Pin_a11)
- net +DIVIDE_OP: now reaches J278.a6 (Pin_a6)
- net -RESET_D_SPD_GATE: now reaches J278.a9 (Pin_a9)
- net +DBL_WORD_ADDRESSING: now reaches J278.b1 (Pin_b1)
- net -STX_E1_NOT_TAG_00: now reaches J278.b11 (Pin_b11)
- net -IA_CYCLE: now reaches J278.b12 (Pin_b12)
- net -DIVIDE_E: now reaches J278.b4 (Pin_b4)
- net -AND_SPD_GATE: now reaches J278.b5 (Pin_b5)
- net -AND_SPD_GATE: now also J340.a3 (Pin_a3)
- net -DC_RESET_1: now reaches J278.b6 (Pin_b6)
- net +STORE_STATUS_E: now reaches J271.a12 (Pin_a12)
- net -INDEX_INSTR: now reaches J271.a4 (Pin_a4)
- net +BR_OR_SKIP_ON_COND: now reaches J271.a7 (Pin_a7)
- net -BSI_E: now reaches J271.a8 (Pin_a8)
- net +FORMAT_5: now reaches J271.a9 (Pin_a9)
- net -LDX_OP: now reaches J271.b1 (Pin_b1)
- net -MDX_OP: now reaches J271.b10 (Pin_b10)
- net -OP_001X0: now reaches J271.b12 (Pin_b12)
- net +BSI_FORMAT_BSC_FORMAT: now reaches J271.b4 (Pin_b4)
- net -BR_OR_SKIP_ON_COND: now reaches J271.b5 (Pin_b5)
- net +BSI_E: now reaches J271.b8 (Pin_b8)
- net +SHIFT_INSTR: now reaches J272.a1 (Pin_a1)
- net -OP_00110: now reaches J272.a11 (Pin_a11)
- net -SHIFT_RIGHT_OP: now reaches J272.a12 (Pin_a12)
- net -STORE_STATUS_E: now reaches J272.a2 (Pin_a2)
- net -LOAD_STATUS_T4: now reaches J272.a3 (Pin_a3)
- net +STX_OP: now reaches J272.a4 (Pin_a4)
- net -SHIFT_LEFT_OP: now reaches J272.a8 (Pin_a8)
- net -XIO_OP: now reaches J272.b1 (Pin_b1)
- net -OP_BIT_0: now reaches J272.b10 (Pin_b10)
- net +SHIFT_RIGHT_OP: now reaches J272.b4 (Pin_b4)
- net +T_4: now reaches J272.b6 (Pin_b6)
- new net +LDX_OP: J271.b2 (Pin_b2)
Other:
- moved on the sheet: J259, J260, J261, J262, J263, J264, J265, J266, J267, J268, J269, J270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

Commit message: Add labels for cable runs, completed tracing for DN111 from previous commit, decided it would be too much work to go back and route later... Completed DN201 page.
Connections:
- net +3V: no longer J263.b2 (Pin_b2), J264.b2 (Pin_b2), J341.b2 (Pin_b2), J344.b2 (Pin_b2)
- net +6V: no longer J263.a10 (Pin_a10), J264.a10 (Pin_a10), J344.a10 (Pin_a10)
- net +E_CYCLES: now also J312.a8 (Pin_a8)
- net +XIO_OP: now also J312.b4 (Pin_b4), J312.b6 (Pin_b6), J312.b8 (Pin_b8)
- net -3V: no longer J263.a5 (Pin_a5), J264.a5 (Pin_a5), J344.a5 (Pin_a5)
- net -XIO_E: now also J312.a6 (Pin_a6), J326.a6 (Pin_a6)
- net -XIO_E2_R_W: now reaches J312.a1 (Pin_a1)
- net -XIO_E2_R_W: now also J276.a1 (Pin_a1), J287.a3 (Pin_a3), J344.b4 (Pin_b4)
- net +B_BIT_6: now reaches J312.a11 (Pin_a11)
- net +B_BIT_5: now reaches J312.a12 (Pin_a12)
- net +E2_CYCLE: now reaches J312.a2 (Pin_a2)
- net -U_BIT_7: now reaches J312.a3 (Pin_a3)
- net DN201_AL4: now reaches J312.a4 (Pin_a4)
- net DN201_AL4: now also J276.a4 (Pin_a4), J320.b3 (Pin_b3), J325.b4 (Pin_b4), J344.b3 (Pin_b3)
- net +E1_CYCLE: now reaches J312.a7 (Pin_a7)
- net -GATE_SENSE_INHIBIT_STOR_USE: now reaches J312.a9 (Pin_a9)
- net -U_BIT_5: now reaches J312.b1 (Pin_b1)
- net -U_BIT_5: now also J276.b1 (Pin_b1)
- net +XIO_E1: now reaches J312.b10 (Pin_b10)
- net +XIO_E1: now also J320.b4 (Pin_b4)
- net DN201_AE4: now reaches J312.b3 (Pin_b3)
- net DN201_AE4: now also J320.a4 (Pin_a4)
- net DN201_AD4: now reaches J312.b5 (Pin_b5)
- net DN201_AD4: now also J320.b5 (Pin_b5)
- net -U_BIT_6: now reaches J276.a3 (Pin_a3)
- net +NOT_STORAGE_USE: now reaches J325.a2 (Pin_a2)
- net +NOT_STORAGE_USE: now also J320.a1 (Pin_a1)
- net +INTERRUPT_REQUEST: now reaches J325.b12 (Pin_b12)
- net +INTERRUPT_REQUEST: now also J319.b8 (Pin_b8)
- net -XIO_TIME_GATE: now reaches J325.b3 (Pin_b3)
- net -XIO_TIME_GATE: now also J263.a3 (Pin_a3), J326.a7 (Pin_a7), J326.b5 (Pin_b5)
- net -INTERRUPT_REQ_INH_STOR_USE: now reaches J325.b8 (Pin_b8)
- net -CS_LEVELS: now reaches J325.b9 (Pin_b9)
- net DN201_BA6: now reaches J311.a2 (Pin_a2)
- net DN201_BA6: now also J326.b6 (Pin_b6)
- net DN201_AA4: now reaches J311.a7 (Pin_a7)
- net DN201_AA4: now also J319.a9 (Pin_a9)
- net +REQ_INTERRUPT_LVL_5: now reaches J311.b3 (Pin_b3)
- net -PROGRAM_STOP_LATCH: now reaches J311.b4 (Pin_b4)
- net -X_CLOCK_ADV_SAMPLE: now reaches J311.b5 (Pin_b5)
- net +PHASE_A: now reaches J311.b8 (Pin_b8)
- net +INT_RUN_MODE: now reaches J264.a4 (Pin_a4)
- net +INT_RUN_MODE: now also J319.b4 (Pin_b4)
- net +STORAGE_USE: now reaches J320.a3 (Pin_a3)
- net -CS_LEVEL_1: now reaches J319.a11 (Pin_a11)
- net -INTERRUPT_LVLS_0123: now reaches J319.a2 (Pin_a2)
- net -CS_LEVEL_0: now reaches J319.b10 (Pin_b10)
- net -INTERRUPT_REQUESTS_23: now reaches J319.b11 (Pin_b11)
- net -INTERRUPT_REQUESTS_45: now reaches J319.b12 (Pin_b12)
- net DN201_AG4: now reaches J319.b3 (Pin_b3)
- net DN201_AG4: now also J326.a12 (Pin_a12)
- net -INTERRUPT_LVLS_45: now reaches J319.b5 (Pin_b5)
- net -INTERRUPT_REQUESTS_01: now reaches J319.b9 (Pin_b9)
- net -INTERRUPT_LEVEL_5: now reaches J326.a11 (Pin_a11)
- net -CCC_DECREM_SAMPLE: now reaches J326.a4 (Pin_a4)
- net -T_7: now reaches J326.a9 (Pin_a9)
- net -DC_RESET_2: now reaches J326.b10 (Pin_b10)
- net -DC_RESET_2: now also J326.b9 (Pin_b9)
- net -T_5: now reaches J326.b11 (Pin_b11)
- net -RESET_INTERRUPT_LVLS_SP: now reaches J326.b12 (Pin_b12)
- net +XIO_E2_R_W: now reaches J287.a1 (Pin_a1)
Other:
- note added: "5800000"
- note added: "5800002"
- note added: "5800236"
- note added: "5800238"
- note added: "5800509"
- note added: "5803421"
- note added: "5803794"
- note added: "5804675"
- note added: "5804676"
- note added: "CABL 01A-C1N4"
- note added: "CABL 01A-C1N6"
- note added: "CABL 01B-B1A3"
- note added: "CABL 01B-B1A4"
- note added: "CABL 01B-B1A7"

Commit message: Add labels for bottom T[x] connectors, finished page DU101.
Connections:
- net +ENTRY_GATE: now reaches J263.a4 (Pin_a4)
Other:
- moved on the sheet: J290, J298, J306, J314

Commit message: Finish page KA101-KA111
Connections:
- net -DC_RESET_2 is gone; now on net -DC_RESET_1: J326.b10 (Pin_b10), J326.b9 (Pin_b9)
- net +3V: no longer J262.b2 (Pin_b2)
- net +6V: no longer J262.a10 (Pin_a10)
- net +PHASE_A: now also J274.b4 (Pin_b4)
- net -3V: no longer J262.a5 (Pin_a5)
- net -ARITH_CTRL_B: now also J274.a4 (Pin_a4)
- net -CS_LEVELS: now also J274.a8 (Pin_a8)
- net -DC_RESET_1: now also J263.a9 (Pin_a9), J273.b6 (Pin_b6), J341.a6 (Pin_a6)
- net -T_7: now also J274.a3 (Pin_a3)
- net KA111_BL4: now reaches J281.a6 (Pin_a6)
- net KA111_BL4: now also J273.b5 (Pin_b5)
- net -PARITY_STOP: now reaches J281.a8 (Pin_a8)
- net +PROG_START_KEY_2: now reaches J281.b6 (Pin_b6)
- net +SGL_STEP_MODE: now reaches J262.b12 (Pin_b12)
- net +SGL_STEP_MODE: now also J274.b6 (Pin_b6)
- net -RESET_KEY: now reaches J262.b9 (Pin_b9)
- net -RESET_KEY: now also J273.b10 (Pin_b10)
- net KA101_AA5: now reaches J286.a12 (Pin_a12)
- net KA101_AA5: now also J286.a4 (Pin_a4)
- net KA101_AA3: now reaches J286.a3 (Pin_a3)
- net KA101_AA3: now also J274.a12 (Pin_a12)
- net KA101_AA4: now reaches J286.a9 (Pin_a9)
- net KA101_AA4: now also J274.b10 (Pin_b10)
- net -PHASE_A_SP_A: now reaches J273.a1 (Pin_a1)
- net -PHASE_A_SP_A: now also J340.b2 (Pin_b2)
- net -BRANCH_2: now reaches J273.a11 (Pin_a11)
- net -SH_RT_ROT_16_48: now reaches J273.a12 (Pin_a12)
- net -START_ADVANCE: now reaches J273.a3 (Pin_a3)
- net +RUN_PROG_LOAD_DOT_ON_RUN: now reaches J273.a6 (Pin_a6)
- net +RUN_PROG_LOAD_DOT_ON_RUN: now also J263.b6 (Pin_b6)
- net -BRANCH_1: now reaches J273.a9 (Pin_a9)
- net -T_CLOCK_ADV_SP: now reaches J273.b1 (Pin_b1)
- net -INTERRUPT_REQUEST: now reaches J273.b11 (Pin_b11)
- net +OSC_TGR: now reaches J273.b12 (Pin_b12)
- net -DELAY: now reaches J273.b4 (Pin_b4)
- net +CPU_STOP_LATCH: now reaches J273.b8 (Pin_b8)
- net -POWER_ON_RESET: now reaches J273.b9 (Pin_b9)
- net +PHASE_B: now reaches J264.b5 (Pin_b5)
- net +PHASE_B: now also J274.b9 (Pin_b9)
- net -SINGLE_STORAGE_CYCLE: now reaches J274.a1 (Pin_a1)
- net -SET_INTERRUPT_SP: now reaches J274.a11 (Pin_a11)
- net -T_CLK_ADV_SAMPLE: now reaches J274.a2 (Pin_a2)
- net -WAIT_NOT_STRG_LOAD_DISPL: now reaches J274.a6 (Pin_a6)
- net -SINGLE_INSTRUCTION: now reaches J274.a7 (Pin_a7)
- net +T_7: now reaches J274.a9 (Pin_a9)
- net -OSC_TGR: now reaches J274.b11 (Pin_b11)
- net -T7_COUNT_0: now reaches J274.b12 (Pin_b12)
- net -SHIFT_CTRL: now reaches J274.b5 (Pin_b5)
- net -CPU_STOP_LATCH: now reaches J274.b8 (Pin_b8)
Other:
- note added: "5803765"
- note added: "5806213"
- note added: "CABL ZK111"
- note added: "DOT A"
- note added: "DOT OR"

Commit message: Finish page KB101-KB111
Connections:
- net +3V: no longer J339.b2 (Pin_b2)
- net +6V: no longer J339.a10 (Pin_a10)
- net +BR_OR_SKIP_ON_COND: now also J322.b9 (Pin_b9)
- net +BSI_FORMAT_BSC_FORMAT: now also J321.b4 (Pin_b4)
- net +E_CYCLES: now also J275.a11 (Pin_a11)
- net +FORMAT_5: now also J322.b10 (Pin_b10)
- net +LDX_OP: now also J322.b6 (Pin_b6)
- net +PHASE_A: now also J321.b10 (Pin_b10)
- net +PHASE_B: now also J322.a1 (Pin_a1)
- net -3V: no longer J339.a5 (Pin_a5)
- net -BRANCH_1: now also J321.b12 (Pin_b12)
- net -BRANCH_2: now also J322.a2 (Pin_a2)
- net -CS_LEVELS: now also J321.b8 (Pin_b8)
- net -DC_RESET_1: now also J321.a1 (Pin_a1)
- net -PHASE_A_SP_A: now also J322.b12 (Pin_b12)
- net -SHIFT_CTRL: now also J321.b6 (Pin_b6)
- net -M_TO_I_SPD_SAMPLE: now reaches J339.a6 (Pin_a6)
- net -M_TO_I_SPD_SAMPLE: now also J321.b5 (Pin_b5)
- net -A_TO_M_SPD_SAMPLE: now reaches J339.a7 (Pin_a7)
- net -A_TO_M_SPD_SAMPLE: now also J321.a8 (Pin_a8)
- net -FORMAT_5: now reaches J322.a11 (Pin_a11)
- net +T_5: now reaches J322.a12 (Pin_a12)
- net -ADD_TO_STOR_SET_INTLK_SPL: now reaches J322.a3 (Pin_a3)
- net -T_1: now reaches J322.a4 (Pin_a4)
- net -ADD_TO_STOR_INTLK: now reaches J322.a6 (Pin_a6)
- net +MDX: now reaches J322.a7 (Pin_a7)
- net +TAG_00: now reaches J322.a9 (Pin_a9)
- net -E_GT_TURN_ON: now reaches J322.b1 (Pin_b1)
- net +MOD_9: now reaches J322.b11 (Pin_b11)
- net +ADD_TO_STORAGE_OP: now reaches J322.b3 (Pin_b3)
- net -BRANCH_OUT: now reaches J322.b8 (Pin_b8)
- net +T_6: now reaches J275.a12 (Pin_a12)
- net -BR-2_NOT_BR-1_RESET_CCC: now reaches J275.a9 (Pin_a9)
- net -BR-2_NOT_BR-1_RESET_CCC: now also J321.b1 (Pin_b1)
- net +SLC_OP: now reaches J275.b10 (Pin_b10)
- net -BSI_OR_BSC_RESET_OVERFLOW: now reaches J321.a11 (Pin_a11)
- net -SKIP_COND: now reaches J321.a2 (Pin_a2)
- net -BSI_TRUE_OR_BSC_TRUE: now reaches J321.a3 (Pin_a3)
- net -I1_T4: now reaches J321.a4 (Pin_a4)
- net +I1_T4: now reaches J321.a6 (Pin_a6)
- net -ARITH_CTRL_A: now reaches J321.a7 (Pin_a7)
- net +BRANCH_1: now reaches J321.a9 (Pin_a9)
- net +BRANCH_2: now reaches J321.b11 (Pin_b11)
- net -SKIP_SAMPLE: now reaches J321.b3 (Pin_b3)
- net +T7_PWR: now reaches J321.b9 (Pin_b9)
Other:
- note added: "5804623"
- note added: "CABL 01B-B1A2"
