File: 1130_backplane/01B-A1.kicad_sch (KiCad schematic)
At the start: 89 parts

Commit message: Finish page KM301-KM321
Parts:
- added JP?: NO DISK, symbol Jumper:Jumper_2_Bridged
- added JP?: NO 1132, symbol Jumper:Jumper_2_Bridged
Connections:
- net +GATE_INTERRUPT: now also J295.b12 (Pin_b12), J295.b8 (Pin_b8), J303.b12 (Pin_b12), J303.b8 (Pin_b8), J304.b12 (Pin_b12), J304.b8 (Pin_b8)
- net +I2_T6: now also J295.b5 (Pin_b5), J303.b5 (Pin_b5), J304.b5 (Pin_b5)
- net +REQ_INTERRUPT_LVL_0: now also J304.b11 (Pin_b11)
- net -DC_RESET_1: now also J295.a2 (Pin_a2), J303.a2 (Pin_a2), J304.a2 (Pin_a2)
- net -INTERRUPT_LEVEL_1: now also J304.a7 (Pin_a7)
- net -INTERRUPT_LEVEL_3: now also J303.a7 (Pin_a7)
- net -INTERRUPT_LEVEL_5: now also J295.a7 (Pin_a7)
- net -INTERRUPT_LVLS_0123: now also J295.b3 (Pin_b3), J303.a8 (Pin_a8), J304.a8 (Pin_a8)
- net -INTERRUPT_LVLS_45: now also J295.a8 (Pin_a8)
- net -INTERRUPT_REQUESTS_01: now also J304.a3 (Pin_a3)
- net -INTERRUPT_REQUESTS_23: now also J303.a3 (Pin_a3)
- net -INTERRUPT_REQUESTS_45: now also J295.a3 (Pin_a3)
- net -RESET_INTERRUPT_LVLS_SP: now also J295.a9 (Pin_a9), J303.a9 (Pin_a9), J304.a9 (Pin_a9)
- net -SET_INTERRUPT_SP: now also J295.a11 (Pin_a11), J303.a11 (Pin_a11), J304.a11 (Pin_a11)
- net GND: now also JP?.2 (B), JP?.2 (B)
- net +INTERRUPT_LVL_TGR_4: now reaches J295.a1 (Pin_a1)
- net +INTERRUPT_LVL_TGR_4: now also J261.a9 (Pin_a9)
- net -INTERRUPT_LEVEL_4: now reaches J295.a12 (Pin_a12)
- net -INTERRUPT_LEVEL_4: now also J264.a8 (Pin_a8)
- net +CS_LVL_0_PWR: now reaches J295.a4 (Pin_a4)
- net +INTERRUPT_LVL_TGR_5: now reaches J295.b1 (Pin_b1)
- net +INTERRUPT_LVL_TGR_5: now also J261.b10 (Pin_b10)
- net +REG_INTERRUPT_LVL_5: now reaches J295.b10 (Pin_b10)
- net +INTERRUPT_REG_LVL_4: now reaches J295.b11 (Pin_b11)
- net +INTERRUPT_LVL_TGR_2: now reaches J303.a1 (Pin_a1)
- net +INTERRUPT_LVL_TGR_2: now also J261.a8 (Pin_a8)
- net +INTERRUPT_LVL_TGR_3: now reaches J303.b1 (Pin_b1)
- net +INTERRUPT_LVL_TGR_3: now also J261.b9 (Pin_b9)
- net +INTERRUPT_REQ_LVL_3: now reaches J303.b10 (Pin_b10)
- net +INTERRUPT_REQ_LVL_2: now reaches J303.b11 (Pin_b11)
- net +INTERRUPT_REQ_LVL_2: now also JP?.1 (A)
- net -INTERRUPT_LVL_TGR_0: now reaches J303.b3 (Pin_b3)
- net -INTERRUPT_LVL_TGR_0: now also J304.b4 (Pin_b4)
- net -INTERRUPT_LVL_TGR_1: now reaches J303.b6 (Pin_b6)
- net -INTERRUPT_LVL_TGR_1: now also J304.b9 (Pin_b9)
- net +INTERRUPT_LVL_TGR_0: now reaches J261.a7 (Pin_a7)
- net +INTERRUPT_LVL_TGR_0: now also J304.a1 (Pin_a1)
- net +INTERRUPT_LVL_TGR_1: now reaches J261.b8 (Pin_b8)
- net +INTERRUPT_LVL_TGR_1: now also J304.b1 (Pin_b1)
- net +PRINTER_LVL_1_INTERRUPT_REQ: now reaches J304.b10 (Pin_b10)
- net +PRINTER_LVL_1_INTERRUPT_REQ: now also J263.b10 (Pin_b10), JP?.1 (A)
Other:
- note added: "5803761"
- moved on the sheet: JP?

Commit message: Finish page KR101-KR111
Connections:
- net -DC_RESET_1: now also J316.b1 (Pin_b1)
- net -PARITY_STOP: now also J262.b3 (Pin_b3), J264.b10 (Pin_b10), J316.b4 (Pin_b4)
- net -START_ADVANCE: now also J316.b5 (Pin_b5)
- net -T_6: now also J316.a2 (Pin_a2)
- net -X_6: now also J316.a3 (Pin_a3)
- net +CK_BIT_P1: now reaches J260.a6 (Pin_a6)
- net +CK_BIT_P1: now also J316.b12 (Pin_b12), J344.a11 (Pin_a11)
- net +CK_BIT_P2: now reaches J260.b6 (Pin_b6)
- net +CK_BIT_P2: now also J316.b8 (Pin_b8), J342.a11 (Pin_a11)
- net -EVEN_PARITY_1: now reaches J341.a4 (Pin_a4)
- net -EVEN_PARITY_1: now also J316.a8 (Pin_a8)
- net -EVEN_PARITY_2: now reaches J341.a5 (Pin_a5)
- net -EVEN_PARITY_2: now also J316.a9 (Pin_a9)
- net +EVEN_PARITY_1: now reaches J341.b4 (Pin_b4)
- net +EVEN_PARITY_1: now also J316.b10 (Pin_b10)
- net +EVEN_PARITY_2: now reaches J341.b5 (Pin_b5)
- net +EVEN_PARITY_2: now also J316.a6 (Pin_a6)
- net -B_BIT_CK_2: now reaches J297.b10 (Pin_b10)
- net -B_BIT_CK_2: now also J316.a7 (Pin_a7)
- net -B_BIT_CK_1: now reaches J297.b9 (Pin_b9)
- net -B_BIT_CK_1: now also J316.b9 (Pin_b9)
- net KR111_AY6: now reaches J264.b1 (Pin_b1)
- net KR111_AY6: now also J316.b3 (Pin_b3)
- net -SENSE_AMP_BIT_16: now reaches J316.a1 (Pin_a1)
- net -DC_RESET_B_8-15: now reaches J316.a11 (Pin_a11)
- net +STORAGE_WRITE_CYCLE: now reaches J316.a12 (Pin_a12)
- net -SENSE_AMP_BIT_17: now reaches J316.a4 (Pin_a4)
- net +CHK_TGR_CTRL_GATE: now reaches J316.b11 (Pin_b11)
- net +PARITY_RUN_SW: now reaches J316.b6 (Pin_b6)
Other:
- note added: "5803817"
- note added: "CABL 01B-B1T2"
Changed lines of the file:
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@@
     (effects (font (size 5 5) (thickness 1) bold) (justify left bottom))
+  )
+  (text "5803817" (at 543.56 139.7 0)
+    (effects (font (size 1.27 1.27)) (justify left bottom))
   )
   (text "C" (at 323.85 26.67 0)
@@
     (effects (font (size 1.27 1.27)) (justify left bottom))
   )
+  (text "CABL 01B-B1T2" (at 393.7 24.13 0)
+    (effects (font (size 1.27 1.27)) (justify left bottom))
+  )
   (text "E" (at 313.69 379.73 0)
     (effects (font (size 1.27 1.27)) (justify left bottom))
@@
     (effects (font (size 1.27 1.27)) (justify left bottom))
   )
+  (label "+EVEN_PARITY_1" (at 553.72 165.1 0)
+    (effects (font (size 1.27 1.27)) (justify left bottom))
+  )
   (label "+T_2" (at 33.02 160.02 180)
     (effects (font (size 1.27 1.27)) (justify right bottom))
@@
     (effects (font (size 1.27 1.27)) (justify left bottom))
   )
+  (label "+EVEN_PARITY_2" (at 541.02 154.94 180)
+    (effects (font (size 1.27 1.27)) (justify right bottom))
+  )
   (label "+A-REG_EQUAL_0_LATCHED" (at 287.02 109.22 180)
     (effects (font (size 1.27 1.27)) (justify right bottom))
@@
     (effects (font (size 1.27 1.27)) (justify right bottom))
   )
+  (label "-PARITY_STOP" (at 45.72 317.5 0)
+    (effects (font (size 1.27 1.27)) (justify left bottom))
+  )
   (label "-INTERRUPT_REQUESTS_45" (at 553.72 284.48 0)
     (effects (font (size 1.27 1.27)) (justify left bottom))
@@
     (effects (font (size 1.27 1.27)) (justify right bottom))
   )
+  (label "-X_6" (at 541.02 147.32 180)
+    (effects (font (size 1.27 1.27)) (justify right bottom))
+  )
   (label "+I1_POWERED" (at 744.22 190.5 0)
     (effects (font (size 1.27 1.27)) (justify left bottom))
@@
     (effects (font (size 1.27 1.27)) (justify left bottom))
   )
+  (label "+STORAGE_WRITE_CYCLE" (at 541.02 170.18 180)
+    (effects (font (size 1.27 1.27)) (justify right bottom))
+  )
   (label "+NOT_STORAGE_USE" (at 604.52 264.16 180)
     (effects (font (size 1.27 1.27)) (justify right bottom))
@@
     (effects (font (size 1.27 1.27)) (justify right bottom))
   )
+  (label "-B_BIT_CK_2" (at 541.02 157.48 180)
+    (effects (font (size 1.27 1.27)) (justify right bottom))
+  )
   (label "-T_7" (at 604.52 314.96 180)
     (effects (font (size 1.27 1.27)) (justify right bottom))
@@
     (effects (font (size 1.27 1.27)) (justify right bottom))
   )
+  (label "+CK_BIT_P1" (at 795.02 320.04 180)
+    (effects (font (size 1.27 1.27)) (justify right bottom))
+  )
   (label "-3V" (at 596.9 228.6 180)
     (effects (font (size 1.27 1.27)) (justify right bottom))
@@
     (effects (font (size 1.27 1.27)) (justify right bottom))
   )
+  (label "-EVEN_PARITY_2" (at 795.02 190.5 180)
+    (effects (font (size 1.27 1.27)) (justify right bottom))
+  )
   (label "-3V" (at 342.9 228.6 180)
     (effects (font (size 1.27 1.27)) (justify right bottom))
@@
     (effects (font (size 1.27 1.27)) (justify right bottom))
   )
+  (label "-START_ADVANCE" (at 553.72 152.4 0)
+    (effects (font (size 1.27 1.27)) (justify left bottom))
+  )
   (label "DN201_BA6" (at 617.22 307.34 0)
     (effects (font (size 1.27 1.27)) (justify left bottom))
@@
     (effects (font (size 1.27 1.27)) (justify right bottom))
   )
+  (label "-SENSE_AMP_BIT_16" (at 541.02 142.24 180)
+    (effects (font (size 1.27 1.27)) (justify right bottom))
+  )
   (label "KM201_AB4" (at 553.72 312.42 0)
     (effects (font (size 1.27 1.27)) (justify left bottom))
@@
     (effects (font (size 1.27 1.27)) (justify left bottom))
   )
+  (label "KR111_AY6" (at 553.72 147.32 0)
+    (effects (font (size 1.27 1.27)) (justify left bottom))
+  )
   (label "+I1_CYCLE" (at 744.22 154.94 0)
     (effects (font (size 1.27 1.27)) (justify left bottom))
@@
     (effects (font (size 1.27 1.27)) (justify right bottom))
   )
+  (label "-DC_RESET_1" (at 553.72 142.24 0)
+    (effects (font (size 1.27 1.27)) (justify left bottom))
+  )
   (label "+X_3" (at 223.52 236.22 180)
     (effects (font (size 1.27 1.27)) (justify right bottom))
@@
     (effects (font (size 1.27 1.27)) (justify right bottom))
   )
+  (label "-B_BIT_CK_1" (at 407.67 50.8 90)
+    (effects (font (size 1.27 1.27)) (justify left bottom))
+  )
   (label "KM201_AL4" (at 541.02 312.42 180)
     (effects (font (size 1.27 1.27)) (justify right bottom))
@@
     (effects (font (size 1.27 1.27)) (justify right bottom))
   )
+  (label "-SENSE_AMP_BIT_17" (at 541.02 149.86 180)
+    (effects (font (size 1.27 1.27)) (justify right bottom))
+  )
   (label "-INTERRUPT_LEVEL_1" (at 414.02 309.88 180)
     (effects (font (size 1.27 1.27)) (justify right bottom))
@@
     (effects (font (size 1.27 1.27)) (justify left bottom))
   )
+  (label "+CK_BIT_P2" (at 795.02 243.84 180)
+    (effects (font (size 1.27 1.27)) (justify right bottom))
+  )
   (label "GND" (at 624.84 157.48 0)
     (effects (font (size 1.27 1.27)) (justify left bottom))
@@
     (effects (font (size 1.27 1.27)) (justify left bottom))
   )
+  (label "+EVEN_PARITY_2" (at 807.72 190.5 0)
+    (effects (font (size 1.27 1.27)) (justify left bottom))
+  )
   (label "+OP_BIT_0" (at 236.22 109.22 0)
     (effects (font (size 1.27 1.27)) (justify left bottom))
@@
     (effects (font (size 1.27 1.27)) (justify left bottom))
   )
+  (label "+PARITY_RUN_SW" (at 553.72 154.94 0)
+    (effects (font (size 1.27 1.27)) (justify left bottom))
+  )
   (label "-DC_RESET_1" (at 172.72 193.04 0)
     (effects (font (size 1.27 1.27)) (justify left bottom))
@@
     (effects (font (size 1.27 1.27)) (justify right bottom))
   )
+  (label "-PARITY_STOP" (at 45.72 223.52 0)
+    (effects (font (size 1.27 1.27)) (justify left bottom))
+  )
   (label "-DC_RESET_2" (at 350.52 302.26 180)
     (effects (font (size 1.27 1.27)) (justify right bottom))
@@
     (effects (font (size 1.27 1.27)) (justify left bottom))
   )
+  (label "-EVEN_PARITY_1" (at 795.02 187.96 180)
+    (effects (font (size 1.27 1.27)) (justify right bottom))
+  )
   (label "+XIO_E2_R_W" (at 287.02 256.54 180)
     (effects (font (size 1.27 1.27)) (justify right bottom))
@@
     (effects (font (size 1.27 1.27)) (justify left bottom))
   )
+  (label "+CK_BIT_P1" (at 33.02 154.94 180)
+    (effects (font (size 1.27 1.27)) (justify right bottom))
+  )
   (label "-BR_OR_SKIP_ON_COND" (at 172.72 114.3 0)
     (effects (font (size 1.27 1.27)) (justify left bottom))
@@
     (effects (font (size 1.27 1.27)) (justify right bottom))
   )
+  (label "+CHK_TGR_CTRL_GATE" (at 553.72 167.64 0)
+    (effects (font (size 1.27 1.27)) (justify left bottom))
+  )
   (label "-3V" (at 406.4 114.3 180)
     (effects (font (size 1.27 1.27)) (justify right bottom))
@@
     (effects (font (size 1.27 1.27)) (justify left bottom))
   )
+  (label "+EVEN_PARITY_1" (at 807.72 187.96 0)
+    (effects (font (size 1.27 1.27)) (justify left bottom))
+  )
   (label "-M_TO_I_SPD_GATE" (at 807.72 104.14 0)
     (effects (font (size 1.27 1.27)) (justify left bottom))
@@
     (effects (font (size 1.27 1.27)) (justify right bottom))
   )
+  (label "+CK_BIT_P2" (at 45.72 154.94 0)
+    (effects (font (size 1.27 1.27)) (justify left bottom))
+  )
   (label "+INTERRUPT_LVL_TGR_1" (at 45.72 198.12 0)
     (effects (font (size 1.27 1.27)) (justify left bottom))
@@
     (effects (font (size 1.27 1.27)) (justify left bottom))
   )
+  (label "-B_BIT_CK_2" (at 410.21 50.8 90)
+    (effects (font (size 1.27 1.27)) (justify left bottom))
+  )
   (label "-3V" (at 596.9 152.4 180)
     (effects (font (size 1.27 1.27)) (justify right bottom))
@@
     (effects (font (size 1.27 1.27)) (justify left bottom))
   )
+  (label "+CK_BIT_P1" (at 553.72 170.18 0)
+    (effects (font (size 1.27 1.27)) (justify left bottom))
+  )
   (label "-LDX_OP" (at 299.72 121.92 0)
     (effects (font (size 1.27 1.27)) (justify left bottom))
@@
     (effects (font (size 1.27 1.27)) (justify left bottom))
   )
+  (label "-EVEN_PARITY_2" (at 541.02 162.56 180)
+    (effects (font (size 1.27 1.27)) (justify right bottom))
+  )
   (label "+XIO_OP" (at 160.02 129.54 180)
     (effects (font (size 1.27 1.27)) (justify right bottom))
@@
     (effects (font (size 1.27 1.27)) (justify right bottom))
   )
+  (label "-DC_RESET_B_8-15" (at 541.02 167.64 180)
+    (effects (font (size 1.27 1.27)) (justify right bottom))
+  )
   (label "-SET_INTERRUPT_SP" (at 350.52 312.42 180)
     (effects (font (size 1.27 1.27)) (justify right bottom))
@@
     (effects (font (size 1.27 1.27)) (justify left bottom))
   )
+  (label "-T_6" (at 541.02 144.78 180)
+    (effects (font (size 1.27 1.27)) (justify right bottom))
+  )
   (label "+3V" (at 688.34 106.68 0)
     (effects (font (size 1.27 1.27)) (justify left bottom))
@@
     (effects (font (size 1.27 1.27)) (justify right bottom))
   )
+  (label "+CK_BIT_P2" (at 553.72 160.02 0)
+    (effects (font (size 1.27 1.27)) (justify left bottom))
+  )
   (label "+BRANCH_2" (at 731.52 223.52 180)
     (effects (font (size 1.27 1.27)) (justify right bottom))
@@
     (effects (font (size 1.27 1.27)) (justify right bottom))
   )
+  (label "-B_BIT_CK_1" (at 553.72 162.56 0)
+    (effects (font (size 1.27 1.27)) (justify left bottom))
+  )
   (label "+3V" (at 370.84 144.78 0)
     (effects (font (size 1.27 1.27)) (justify left bottom))
@@
     (effects (font (size 1.27 1.27)) (justify left bottom))
   )
+  (label "-PARITY_STOP" (at 553.72 149.86 0)
+    (effects (font (size 1.27 1.27)) (justify left bottom))
+  )
   (label "GND" (at 624.84 119.38 0)
     (effects (font (size 1.27 1.27)) (justify left bottom))
@@
     (effects (font (size 1.27 1.27)) (justify left bottom))
   )
+  (label "-EVEN_PARITY_1" (at 541.02 160.02 180)
+    (effects (font (size 1.27 1.27)) (justify right bottom))
+  )
   (label "+3V" (at 497.84 297.18 0)
     (effects (font (size 1.27 1.27)) (justify left bottom))
@@
     (effects (font (size 1.27 1.27)) (justify left bottom))
   )
+  (label "KR111_AY6" (at 45.72 294.64 0)
+    (effects (font (size 1.27 1.27)) (justify left bottom))
+  )

Commit message: Finish page KS101-KS111
Connections:
- net +A-REG_EQUAL_0_LATCHED: now also J318.b5 (Pin_b5)
- net +ADD_SUB_GT_E: now also J317.a12 (Pin_a12)
- net +DIVIDE_E: now also J317.a9 (Pin_a9)
- net +T7_END_OP: now also J317.b11 (Pin_b11)
- net -ADD_SUB_GATE_E: now also J318.b6 (Pin_b6)
- net -A_REG_EQUAL_ZERO: now also J318.b11 (Pin_b11)
- net -BSI_OR_BSC_RESET_OVERFLOW: now also J317.a6 (Pin_a6)
- net -DBL_PREC_E2: now also J318.a9 (Pin_a9)
- net -DC_RESET_1: now also J318.b9 (Pin_b9)
- net -LOAD_STATUS_T4: now also J317.b12 (Pin_b12)
- net -SET_DIV_OFLO_E1_E2: now also J317.b4 (Pin_b4)
- net -SKIP_COND: now also J317.a7 (Pin_a7)
- net +CARRY: now reaches J261.a4 (Pin_a4)
- net +CARRY: now also J317.b3 (Pin_b3)
- net +TEMP_CARRY: now reaches J261.b3 (Pin_b3)
- net +TEMP_CARRY: now also J318.a4 (Pin_a4)
- net +OVERFLOW: now reaches J261.b5 (Pin_b5)
- net +OVERFLOW: now also J317.a4 (Pin_a4)
- net +D_BIT_14: now reaches J318.a1 (Pin_a1)
- net -SUB_GATE: now reaches J318.a11 (Pin_a11)
- net +DBL_PREC_CARRY: now reaches J318.a12 (Pin_a12)
- net -A_REG_BIT_0_PWR: now reaches J318.a2 (Pin_a2)
- net -T3_SP: now reaches J318.a3 (Pin_a3)
- net +A_BIT_0: now reaches J318.a6 (Pin_a6)
- net -ADD_GATE_A: now reaches J318.a7 (Pin_a7)
- net -DBL_PREC_CARRY: now reaches J318.a8 (Pin_a8)
- net -SLC_RESET_CARRY: now reaches J318.b1 (Pin_b1)
- net +ACC_BIT_15_SHIFT_LT_ENTRY: now reaches J318.b10 (Pin_b10)
- net +A_REG_BIT_0_PWR: now reaches J318.b12 (Pin_b12)
- net -GATE_CCC_TO_A10-A15: now reaches J318.b3 (Pin_b3)
- net -SHIFT_LT_SAMPLE: now reaches J318.b4 (Pin_b4)
- net +D_BIT_15: now reaches J318.b8 (Pin_b8)
- net -U_BIT_0: now reaches J317.a1 (Pin_a1)
- net +OFLO_GATE: now reaches J317.a11 (Pin_a11)
- net -CARRY_TO_ACC: now reaches J317.a2 (Pin_a2)
- net -OVERFLOW_TO_ACC: now reaches J317.a3 (Pin_a3)
- net +STORE_STATUS_E_T2: now reaches J317.a8 (Pin_a8)
- net +D_BIT_12: now reaches J317.b1 (Pin_b1)
- net +DIV_CT_16_SAMPLE: now reaches J317.b10 (Pin_b10)
- net +D_BIT_10: now reaches J317.b5 (Pin_b5)
- net -U_BIT_15: now reaches J317.b6 (Pin_b6)
- net +D_BIT_11: now reaches J317.b8 (Pin_b8)
- net +D_BIT_13: now reaches J317.b9 (Pin_b9)
Other:
- note added: "5804680"

Commit message: Finish page KT101-KT131
Connections:
- net +ADD_SUB_GT_E: now also J302.a2 (Pin_a2)
- net +A_REG_BIT_0_PWR: now also J302.a4 (Pin_a4)
- net +B_BIT_0_LATCHED: now also J302.b3 (Pin_b3)
- net +CCC_COUNT_0: now also J301.b4 (Pin_b4)
- net +DIVIDE_E: now also J301.b9 (Pin_b9), J309.b10 (Pin_b10)
- net +DIVIDE_E1: now also J302.b1 (Pin_b1), J309.b4 (Pin_b4)
- net +E1_CYCLE: now also J301.a3 (Pin_a3)
- net +E_CYCLES: now also J301.b1 (Pin_b1)
- net +LIKE_SIGNS: now also J301.b10 (Pin_b10)
- net +MULT_OP_E: now also J302.a7 (Pin_a7), J310.b11 (Pin_b11)
- net +OP_BIT_3: now also J301.a9 (Pin_a9)
- net +T_2: now also J301.a7 (Pin_a7)
- net +T_3: now also J302.b12 (Pin_b12)
- net +WRITE_GATE_PHASE_B: now also J310.b8 (Pin_b8)
- net -ARITH_CTRL_A: now also J309.a12 (Pin_a12)
- net -ARITH_CTRL_B: now also J309.b3 (Pin_b3)
- net -A_REG_BIT_0_PWR: now also J302.b5 (Pin_b5)
- net -A_REG_EQUAL_ZERO: now also J310.a12 (Pin_a12)
- net -B_BIT_0_LATCHED: now also J302.b11 (Pin_b11), J309.a1 (Pin_a1)
- net -CCC_COUNT_0: now also J301.a12 (Pin_a12), J309.a4 (Pin_a4)
- net -DBL_PREC_CARRY: now also J309.b5 (Pin_b5)
- net -DIVIDE_E: now also J309.a6 (Pin_a6)
- net -MULTIPLY_E: now also J310.b12 (Pin_b12)
- net -SET_DIV_OFLO_E1_E2: now also J309.a7 (Pin_a7)
- net -SHIFT_CTRL: now also J310.a6 (Pin_a6)
- net -SH_RT_ROT_16_48: now also J310.b4 (Pin_b4)
- net -T3_SP: now also J301.b8 (Pin_b8), J310.a8 (Pin_a8)
- net -T_1: now also J302.a8 (Pin_a8)
- net -T_2: now also J310.a9 (Pin_a9)
- net -DIV_LOAD_Q-15: now reaches J341.b8 (Pin_b8)
- net -DIV_LOAD_Q-15: now also J301.a8 (Pin_a8)
- net +T3_SAMPLE: now reaches J310.a1 (Pin_a1)
- net -SHIFT_RT_SAMPLE: now reaches J310.a11 (Pin_a11)
- net -SLC_BIT: now reaches J310.a2 (Pin_a2)
- net -SET_ARITH_CONTROL: now reaches J310.a3 (Pin_a3)
- net -SHIFT_OP_GATE_T3: now reaches J310.a4 (Pin_a4)
- net -E_NOT_MULT_E1: now reaches J310.a7 (Pin_a7)
- net -E_NOT_MULT_E1: now also J301.a6 (Pin_a6)
- net +CCC_COUNT_0_OR_1: now reaches J310.b1 (Pin_b1)
- net +CCC_COUNT_0_OR_1: now also J302.a1 (Pin_a1)
- net -DC_RESET_OP_REG_AND_OP_FLAGS: now reaches J310.b10 (Pin_b10)
- net -DC_RESET_OP_REG_AND_OP_FLAGS: now also J302.a12 (Pin_a12)
- net -START_MPY_ARITH_ACTION: now reaches J310.b3 (Pin_b3)
- net -START_MPY_ARITH_ACTION: now also J302.a6 (Pin_a6)
- net +ARITH_CTRL: now reaches J310.b5 (Pin_b5)
- net +ARITH_CTRL: now also J261.a2 (Pin_a2)
- net -TURN_OF_SHIFT_CTRL: now reaches J310.b6 (Pin_b6)
- net +SHIFT_CTRL: now reaches J310.b9 (Pin_b9)
- net +SHIFT_CTRL: now also J261.a3 (Pin_a3)
- net +ADD: now reaches J261.a1 (Pin_a1)
- net +ADD: now also J301.b5 (Pin_b5)
- net +ARITH_SIGN: now reaches J261.b1 (Pin_b1)
- net +ARITH_SIGN: now also J302.b9 (Pin_b9), J309.b1 (Pin_b1)
- net +ZERO_REMAINDER: now reaches J261.b4 (Pin_b4)
- net +ZERO_REMAINDER: now also J309.a11 (Pin_a11)
- net -CCC_COUNT_0_OR_1: now reaches J301.a11 (Pin_a11)
- net -QUOT_CORR_SET_D-15: now reaches J301.a2 (Pin_a2)
- net -ADD: now reaches J301.a4 (Pin_a4)
- net +Q_BIT_14: now reaches J301.b11 (Pin_b11)
- net +E_NOT_MULT_E1: now reaches J301.b12 (Pin_b12)
- net -ZERO_REMAINDER: now reaches J301.b3 (Pin_b3)
- net -ZERO_REMAINDER: now also J309.a2 (Pin_a2)
- net -DIVIDE_E1: now reaches J301.b6 (Pin_b6)
- net -ARITH_SIGN: now reaches J302.a9 (Pin_a9)
- net -Q_BIT_15_PWR: now reaches J302.b4 (Pin_b4)
- net +Q_BIT_15: now reaches J302.b6 (Pin_b6)
- net -MULT_D_REG_EQUAL_0: now reaches J302.b8 (Pin_b8)
- net -SHIFT_LT_SPD_SAMPLE_B: now reaches J309.a8 (Pin_a8)
- net -RESET_ACC: now reaches J309.a9 (Pin_a9)
- net -Q_BIT_0_PWR: now reaches J309.b11 (Pin_b11)
- net +REM_OK: now reaches J309.b12 (Pin_b12)
- net +D_REG_EQUAL_ZERO_CKT_1: now reaches J309.b6 (Pin_b6)
- net +T3_PHASE_B: now reaches J309.b8 (Pin_b8)
- net -RESET_A_REG: now reaches J309.b9 (Pin_b9)
Other:
- note added: "5804607"
- note added: "5804616"
