File: 1130_backplane/01B-B1.kicad_sch (KiCad schematic)
At the start: 86 parts

Commit message: Finish page KG101-KG151
Connections:
- net -AND_SPD_GATE: now also J378.a6 (Pin_a6)
- net -A_TO_M_SPD_SAMPLE: now also J376.a4 (Pin_a4), J386.a4 (Pin_a4)
- net -M_TO_I_SPD_SAMPLE: now also J376.a8 (Pin_a8), J386.a8 (Pin_a8)
- net -PHASE_A_SP_A: now also J386.b12 (Pin_b12)
- net GND: now also J377.a1 (Pin_a1), J377.a6 (Pin_a6), J378.a1 (Pin_a1), J387.a1 (Pin_a1), J387.a6 (Pin_a6), J388.a1 (Pin_a1), J388.a6 (Pin_a6)
- net -I_O_TO_B_SP_0-7: now reaches J347.a8 (Pin_a8)
- net -I_O_TO_B_SP_0-7: now also J377.a11 (Pin_a11)
- net +PHASE_B: now reaches J395.a1 (Pin_a1)
- net -RESET_D_SPD_GATE: now reaches J395.a3 (Pin_a3)
- net -RESET_D_REG_SP: now reaches J395.b1 (Pin_b1)
- net -RESET_D_REG_SP: now also J346.b3 (Pin_b3)
- net -I_TO_B_SPD_GATE: now reaches J376.a1 (Pin_a1)
- net -I_TO_B_SPD_GATE: now also J386.a1 (Pin_a1)
- net -I_TO_M_SP_0-7: now reaches J376.a11 (Pin_a11)
- net -A_TO_B_SP_0-7: now reaches J376.a2 (Pin_a2)
- net -PHASE_A_SP_B: now reaches J376.a3 (Pin_a3)
- net -PHASE_A_SP_B: now also J377.b11 (Pin_b11), J377.b8 (Pin_b8), J378.a9 (Pin_a9), J386.a3 (Pin_a3), J386.a7 (Pin_a7), J386.a9 (Pin_a9), J387.b11 (Pin_b11), J387.b8 (Pin_b8)
- net -A_TO_B_0-7_SPD_GATE: now reaches J376.a6 (Pin_a6)
- net -CLOCK_ADV_SP_B: now reaches J376.a7 (Pin_a7)
- net -CLOCK_ADV_SP_B: now also J376.b11 (Pin_b11), J376.b4 (Pin_b4), J376.b8 (Pin_b8), J386.b11 (Pin_b11), J386.b4 (Pin_b4), J386.b8 (Pin_b8)
- net -A_TO_M_SPD_GATE: now reaches J376.b1 (Pin_b1)
- net -A_TO_M_SPD_GATE: now also J386.b1 (Pin_b1)
- net -M_TO_I_SP_0-7: now reaches J376.b10 (Pin_b10)
- net -CLOCK_ADVANCE_SP_A: now reaches J376.b12 (Pin_b12)
- net -A_TO_M_SP_0-7: now reaches J376.b3 (Pin_b3)
- net -M_TO_I_SPD_GATE: now reaches J376.b5 (Pin_b5)
- net -M_TO_I_SPD_GATE: now also J386.b5 (Pin_b5)
- net -I_TO_B_SP_0-7: now reaches J376.b6 (Pin_b6)
- net -I_TO_M_SPD_GATE: now reaches J376.b9 (Pin_b9)
- net -I_TO_M_SPD_GATE: now also J386.b9 (Pin_b9)
- net -I_O_TO_B_SP_8-15: now reaches J387.a11 (Pin_a11)
- net -I_O_ENTR_SAMPLE: now reaches J387.a12 (Pin_a12)
- net -I_O_ENTR_SAMPLE: now also J377.a12 (Pin_a12)
- net -EXCHANGE_A_AND_Q_SP_8-11: now reaches J387.a2 (Pin_a2)
- net -EXCHG_A_AND_Q_SPD_SAMPLE: now reaches J387.a3 (Pin_a3)
- net -EXCHG_A_AND_Q_SPD_SAMPLE: now also J377.a3 (Pin_a3), J377.a9 (Pin_a9), J387.a9 (Pin_a9)
- net -SHIFT_LT_SPD_SAMPLE_B: now reaches J387.a4 (Pin_a4)
- net -SHIFT_LT_SPD_SAMPLE_B: now also J377.a4 (Pin_a4), J378.a4 (Pin_a4), J388.a4 (Pin_a4)
- net -A_TO_U_SP_8-15: now reaches J387.a7 (Pin_a7)
- net -MOD_8: now reaches J387.b1 (Pin_b1)
- net -MOD_8: now also J377.b1 (Pin_b1)
- net -B_TO_I_SP_8-15: now reaches J387.b10 (Pin_b10)
- net -A_TO_U_SPD_SAMPLE: now reaches J387.b12 (Pin_b12)
- net -A_TO_U_SPD_SAMPLE: now also J377.b12 (Pin_b12)
- net -SHIFT_LEFT_Q_SP_8-15: now reaches J387.b3 (Pin_b3)
- net -SHIFT_LT_SPD_SAMPLE_A: now reaches J387.b4 (Pin_b4)
- net -SHIFT_LT_SPD_SAMPLE_A: now also J377.b4 (Pin_b4), J378.b4 (Pin_b4), J388.b4 (Pin_b4), J388.b6 (Pin_b6)
- net -B_TO_I_GATE: now reaches J387.b5 (Pin_b5)
- net -B_TO_I_GATE: now also J377.b5 (Pin_b5)
- net -EXCHANGE_A_AND_Q_SP_12-15: now reaches J387.b6 (Pin_b6)
- net -LOAD_SAMPLE_GATE: now reaches J387.b9 (Pin_b9)
- net -LOAD_SAMPLE_GATE: now also J377.b9 (Pin_b9)
- net -SHIFT_RIGHT_Q_SP_0-7: now reaches J378.a11 (Pin_a11)
- net -AND_SP: now reaches J378.a2 (Pin_a2)
- net -SHIFT_RT_SAMPLE: now reaches J378.a3 (Pin_a3)
- net -U_TO_A_SP_0-7: now reaches J378.a7 (Pin_a7)
- net KG151_AP2: now reaches J378.a8 (Pin_a8)
- net KG151_AP2: now also J378.b11 (Pin_b11), J378.b6 (Pin_b6), J388.a8 (Pin_a8), J388.b11 (Pin_b11)
- net -SHIFT_RIGHT_A_SP_0-7: now reaches J378.b10 (Pin_b10)
- net -U_TO_A_SPD_SAMPLE: now reaches J378.b12 (Pin_b12)
- net -U_TO_A_SPD_SAMPLE: now also J388.b12 (Pin_b12)
- net -SHIFT_LEFT_A_SP_0-7: now reaches J378.b3 (Pin_b3)
- net -SHIFT_RT_Q_SPD_GT: now reaches J378.b9 (Pin_b9)
- net -SHIFT_RT_Q_SPD_GT: now also J388.b9 (Pin_b9)
- net -SHIFT_RIGHT_Q_SP_8-15: now reaches J388.a11 (Pin_a11)
- net -START_IAR_INCREMENT: now reaches J388.a2 (Pin_a2)
- net -SHIFT_LT_SAMPLE: now reaches J388.a3 (Pin_a3)
- net -U_TO_A_SP_8-15: now reaches J388.a7 (Pin_a7)
- net -INC_IAR_SAMPLE: now reaches J388.a9 (Pin_a9)
- net -SHIFT_RIGHT_A_SP_8-15: now reaches J388.b10 (Pin_b10)
- net -SHIFT_LEFT_A_SP_8-15: now reaches J388.b3 (Pin_b3)
- net -I_TO_M_SP_8-15: now reaches J386.a11 (Pin_a11)
- net -A_TO_B_SP_8-15: now reaches J386.a2 (Pin_a2)
- net -A_TO_B_8-15_SPD_GATE: now reaches J386.a6 (Pin_a6)
- net -M_TO_I_SP_8-15: now reaches J386.b10 (Pin_b10)
- net -A_TO_M_SP_8-15: now reaches J386.b3 (Pin_b3)
- net -I_TO_B_SP_8-15: now reaches J386.b6 (Pin_b6)
- net -EXCHANGE_A_AND_Q_SP_0-3: now reaches J377.a2 (Pin_a2)
- net -A_TO_U_SP_0-7: now reaches J377.a7 (Pin_a7)
- net -B_TO_I_SP_0-7: now reaches J377.b10 (Pin_b10)
- net -SHIFT_LEFT_Q_SP_0-7: now reaches J377.b3 (Pin_b3)
- net -EXCHANGE_A_AND_Q_SP_4-7: now reaches J377.b6 (Pin_b6)
Other:
- note added: "5806207"

Commit message: Finish page KG201-KG111
Connections:
- net -A_TO_M_SPD_GATE: now also J346.b1 (Pin_b1)
- net -B_TO_I_GATE: now also J345.b5 (Pin_b5)
- net -INC_IAR_SAMPLE: now also J345.b6 (Pin_b6)
- net -I_TO_M_SPD_GATE: now also J346.b8 (Pin_b8)
- net -M_TO_I_SPD_GATE: now also J345.b1 (Pin_b1)
- net -IAR_0-7_INCR_GT: now reaches J345.a2 (Pin_a2)
- net -IAR_8-15_INCR_GT: now reaches J345.b2 (Pin_b2)
- net +I_BIT_13: now reaches J421.a12 (Pin_a12)
- net +I_BIT_12: now reaches J421.a4 (Pin_a4)
- net +I_BIT_7: now reaches J421.a6 (Pin_a6)
- net +I_BIT_6: now reaches J421.a7 (Pin_a7)
- net +I_BIT_5: now reaches J421.a8 (Pin_a8)
- net +I_BIT_4: now reaches J421.a9 (Pin_a9)
- net +I_BIT_14: now reaches J421.b10 (Pin_b10)
- net -INCR_11_SAMPLE: now reaches J421.b11 (Pin_b11)
- net -INCR_3_SAMPLE: now reaches J421.b12 (Pin_b12)
- net -INCR_7_SAMPLE: now reaches J421.b3 (Pin_b3)
- net +I_BIT_8: now reaches J421.b4 (Pin_b4)
- net +I_BIT_9: now reaches J421.b5 (Pin_b5)
- net +I_BIT_10: now reaches J421.b6 (Pin_b6)
- net +I_BIT_11: now reaches J421.b8 (Pin_b8)
- net +I_BIT_15: now reaches J421.b9 (Pin_b9)
Other:
- note added: "5803807"
Changed lines of the file:
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@@
-    (effects (font (size 5 5) (thickness 1) bold) (justify left bottom))
-  )
-  (text "4" (at 316.23 198.12 0)
     (effects (font (size 5 5) (thickness 1) bold) (justify left bottom))
   )
@@
     (effects (font (size 1.27 1.27)) (justify left bottom))
   )
-  (text "3" (at 316.23 160.02 0)
-    (effects (font (size 5 5) (thickness 1) bold) (justify left bottom))
-  )
   (text "10" (at 21.59 63.5 0)
     (effects (font (size 1.27 1.27)) (justify left bottom))
@@
     (effects (font (size 1.27 1.27)) (justify left bottom))
   )
-  (text "5" (at 316.23 236.22 0)
-    (effects (font (size 5 5) (thickness 1) bold) (justify left bottom))
-  )
   (text "T2" (at 397.51 33.02 0)
     (effects (font (size 5 5) (thickness 1) bold) (justify left bottom))
@@
     (effects (font (size 5 5) (thickness 1) bold) (justify left bottom))
   )
+  (text "5803807" (at 734.06 177.8 0)
+    (effects (font (size 1.27 1.27)) (justify left bottom))
+  )
   (text "3" (at 833.12 160.02 0)
     (effects (font (size 5 5) (thickness 1) bold) (justify left bottom))
@@
     (effects (font (size 1.27 1.27)) (justify left bottom))
   )
+  (label "-INCR_7_SAMPLE" (at 744.22 185.42 0)
+    (effects (font (size 1.27 1.27)) (justify left bottom))
+  )
   (label "-IO_BIT_3" (at 744.22 223.52 0)
     (effects (font (size 1.27 1.27)) (justify left bottom))
@@
     (effects (font (size 1.27 1.27)) (justify left bottom))
   )
+  (label "-IAR_0-7_INCR_GT" (at 33.02 106.68 180)
+    (effects (font (size 1.27 1.27)) (justify right bottom))
+  )
   (label "-3V" (at 279.4 190.5 180)
     (effects (font (size 1.27 1.27)) (justify right bottom))
@@
     (effects (font (size 1.27 1.27)) (justify left bottom))
   )
+  (label "+I_BIT_14" (at 744.22 203.2 0)
+    (effects (font (size 1.27 1.27)) (justify left bottom))
+  )
   (label "-U_TO_A_SP_0-7" (at 350.52 233.68 180)
     (effects (font (size 1.27 1.27)) (justify right bottom))
@@
     (effects (font (size 1.27 1.27)) (justify right bottom))
   )
+  (label "+I_BIT_13" (at 731.52 208.28 180)
+    (effects (font (size 1.27 1.27)) (justify right bottom))
+  )
   (label "-3V" (at 533.4 304.8 180)
     (effects (font (size 1.27 1.27)) (justify right bottom))
@@
     (effects (font (size 1.27 1.27)) (justify right bottom))
   )
+  (label "+I_BIT_9" (at 744.22 190.5 0)
+    (effects (font (size 1.27 1.27)) (justify left bottom))
+  )
   (label "-3V" (at 88.9 304.8 180)
     (effects (font (size 1.27 1.27)) (justify right bottom))
@@
     (effects (font (size 1.27 1.27)) (justify left bottom))
   )
+  (label "+I_BIT_5" (at 731.52 198.12 180)
+    (effects (font (size 1.27 1.27)) (justify right bottom))
+  )
   (label "-IO_BIT_13" (at 852.17 234.95 0)
     (effects (font (size 1.27 1.27)) (justify left bottom))
@@
     (effects (font (size 1.27 1.27)) (justify left bottom))
   )
+  (label "+I_BIT_7" (at 731.52 193.04 180)
+    (effects (font (size 1.27 1.27)) (justify right bottom))
+  )
   (label "+3V" (at 751.84 297.18 0)
     (effects (font (size 1.27 1.27)) (justify left bottom))
   )
+  (label "+I_BIT_12" (at 731.52 187.96 180)
+    (effects (font (size 1.27 1.27)) (justify right bottom))
+  )
   (label "+3V" (at 307.34 220.98 0)
     (effects (font (size 1.27 1.27)) (justify left bottom))
@@
     (effects (font (size 1.27 1.27)) (justify left bottom))
   )
+  (label "+I_BIT_6" (at 731.52 195.58 180)
+    (effects (font (size 1.27 1.27)) (justify right bottom))
+  )
   (label "+6V" (at 323.85 58.42 180)
     (effects (font (size 1.27 1.27)) (justify right bottom))
@@
     (effects (font (size 1.27 1.27)) (justify right bottom))
   )
+  (label "+I_BIT_4" (at 731.52 200.66 180)
+    (effects (font (size 1.27 1.27)) (justify right bottom))
+  )
   (label "GND" (at 561.34 309.88 0)
     (effects (font (size 1.27 1.27)) (justify left bottom))
@@
     (effects (font (size 1.27 1.27)) (justify right bottom))
   )
+  (label "-M_TO_I_SPD_GATE" (at 45.72 104.14 0)
+    (effects (font (size 1.27 1.27)) (justify left bottom))
+  )
   (label "-I_O_ENTR_SAMPLE" (at 350.52 208.28 180)
     (effects (font (size 1.27 1.27)) (justify right bottom))
@@
     (effects (font (size 1.27 1.27)) (justify left bottom))
   )
+  (label "-IAR_8-15_INCR_GT" (at 45.72 106.68 0)
+    (effects (font (size 1.27 1.27)) (justify left bottom))
+  )
   (label "-3V" (at 279.4 152.4 180)
     (effects (font (size 1.27 1.27)) (justify right bottom))
@@
     (effects (font (size 1.27 1.27)) (justify left bottom))
   )
+  (label "-A_TO_M_SPD_GATE" (at 45.72 142.24 0)
+    (effects (font (size 1.27 1.27)) (justify left bottom))
+  )
   (label "+6V" (at 469.9 317.5 180)
     (effects (font (size 1.27 1.27)) (justify right bottom))
@@
     (effects (font (size 1.27 1.27)) (justify right bottom))
   )
+  (label "-I_TO_M_SPD_GATE" (at 45.72 160.02 0)
+    (effects (font (size 1.27 1.27)) (justify left bottom))
+  )
   (label "+6V" (at 215.9 317.5 180)
     (effects (font (size 1.27 1.27)) (justify right bottom))
@@
     (effects (font (size 1.27 1.27)) (justify left bottom))
   )
+  (label "-INCR_11_SAMPLE" (at 744.22 205.74 0)
+    (effects (font (size 1.27 1.27)) (justify left bottom))
+  )
   (label "-SHIFT_RIGHT_A_SP_8-15" (at 426.72 241.3 0)
     (effects (font (size 1.27 1.27)) (justify left bottom))
@@
     (effects (font (size 1.27 1.27)) (justify right bottom))
   )
+  (label "-INCR_3_SAMPLE" (at 744.22 208.28 0)
+    (effects (font (size 1.27 1.27)) (justify left bottom))
+  )
   (label "-3V" (at 723.9 114.3 180)
     (effects (font (size 1.27 1.27)) (justify right bottom))
@@
     (effects (font (size 1.27 1.27)) (justify right bottom))
   )
+  (label "+I_BIT_11" (at 744.22 198.12 0)
+    (effects (font (size 1.27 1.27)) (justify left bottom))
+  )
   (label "+3V" (at 751.84 182.88 0)
     (effects (font (size 1.27 1.27)) (justify left bottom))
@@
     (effects (font (size 1.27 1.27)) (justify left bottom))
   )
+  (label "-INC_IAR_SAMPLE" (at 45.72 116.84 0)
+    (effects (font (size 1.27 1.27)) (justify left bottom))
+  )
   (label "+3V" (at 688.34 220.98 0)
     (effects (font (size 1.27 1.27)) (justify left bottom))
@@
     (effects (font (size 1.27 1.27)) (justify right bottom))
   )
+  (label "+I_BIT_10" (at 744.22 193.04 0)
+    (effects (font (size 1.27 1.27)) (justify left bottom))
+  )
+  (label "+I_BIT_15" (at 744.22 200.66 0)
+    (effects (font (size 1.27 1.27)) (justify left bottom))
+  )
   (label "-3V" (at 152.4 152.4 180)
     (effects (font (size 1.27 1.27)) (justify right bottom))
   )
+  (label "-B_TO_I_GATE" (at 45.72 114.3 0)
+    (effects (font (size 1.27 1.27)) (justify left bottom))
+  )
   (label "-3V" (at 215.9 228.6 180)
     (effects (font (size 1.27 1.27)) (justify right bottom))
@@
     (effects (font (size 1.27 1.27)) (justify right bottom))
   )
+  (label "+I_BIT_8" (at 744.22 187.96 0)
+    (effects (font (size 1.27 1.27)) (justify left bottom))
+  )
   (label "-IO_BIT_3" (at 807.72 223.52 0)

Commit message: Finish page KG221-KG151
Connections:
- net +3V: no longer J348.b2 (Pin_b2)
- net +6V: no longer J348.a10 (Pin_a10)
- net -3V: no longer J348.a5 (Pin_a5)
- net -A_TO_B_0-7_SPD_GATE: now also J345.a4 (Pin_a4)
- net -A_TO_B_8-15_SPD_GATE: now also J345.b4 (Pin_b4)
- net -A_TO_U_SPD_SAMPLE: now also J348.b1 (Pin_b1)
- net -I_TO_B_SPD_GATE: now also J345.a5 (Pin_a5)
- net -U_TO_A_SPD_SAMPLE: now also J348.a6 (Pin_a6)
- net -DC_SET_D_0-7: now reaches J347.b6 (Pin_b6)
- net +GATE_I_TO_A_0-7: now reaches J345.a3 (Pin_a3)
- net +GATE_I_TO_A_8-15: now reaches J345.b3 (Pin_b3)
- net +GATE_B_TO_D_0-7: now reaches J346.a4 (Pin_a4)
- net +GATE_B_TO_D_8-15: now reaches J346.b4 (Pin_b4)
Other:
- note added: "CABL 01B-A1N5"
Changed lines of the file:
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@@
     (stroke (width 0) (type solid) (color 0 0 0 0))
   )
-  (wire (pts (xy 25.4 228.6) (xy 33.02 228.6))
-    (stroke (width 0) (type default) (color 0 0 0 0))
-  )
   (wire (pts (xy 363.22 259.08) (xy 370.84 259.08))
     (stroke (width 0) (type default) (color 0 0 0 0))
@@
     (stroke (width 0) (type solid) (color 0 0 0 0))
   )
-  (wire (pts (xy 45.72 220.98) (xy 53.34 220.98))
-    (stroke (width 0) (type default) (color 0 0 0 0))
-  )
   (wire (pts (xy 617.22 233.68) (xy 624.84 233.68))
     (stroke (width 0) (type default) (color 0 0 0 0))
@@
     (stroke (width 0) (type solid) (color 0 0 0 0))
   )
-  (wire (pts (xy 25.4 241.3) (xy 33.02 241.3))
-    (stroke (width 0) (type default) (color 0 0 0 0))
-  )
   (polyline (pts (xy 300.99 33.02) (xy 302.26 33.02))
     (stroke (width 0) (type solid) (color 0 0 0 0))
@@
     (effects (font (size 5 5) (thickness 1) bold) (justify left bottom))
   )
+  (text "CABL 01B-A1N5" (at 31.75 215.9 0)
+    (effects (font (size 1.27 1.27)) (justify left bottom))
+  )
   (text "E" (at 299.72 379.73 0)
     (effects (font (size 1.27 1.27)) (justify left bottom))
@@
     (effects (font (size 1.27 1.27)) (justify right bottom))
   )
+  (label "+GATE_B_TO_D_8-15" (at 45.72 149.86 0)
+    (effects (font (size 1.27 1.27)) (justify left bottom))
+  )
   (label "GND" (at 180.34 195.58 0)
     (effects (font (size 1.27 1.27)) (justify left bottom))
@@
     (effects (font (size 1.27 1.27)) (justify left bottom))
   )
+  (label "+GATE_I_TO_A_0-7" (at 33.02 109.22 180)
+    (effects (font (size 1.27 1.27)) (justify right bottom))
+  )
   (label "-3V" (at 406.4 228.6 180)
     (effects (font (size 1.27 1.27)) (justify right bottom))
@@
     (effects (font (size 1.27 1.27)) (justify left bottom))
   )
+  (label "-A_TO_B_0-7_SPD_GATE" (at 33.02 111.76 180)
+    (effects (font (size 1.27 1.27)) (justify right bottom))
+  )
   (label "GND" (at 561.34 157.48 0)
     (effects (font (size 1.27 1.27)) (justify left bottom))
@@
     (effects (font (size 1.27 1.27)) (justify left bottom))
   )
-  (label "-3V" (at 25.4 228.6 180)
-    (effects (font (size 1.27 1.27)) (justify right bottom))
-  )
   (label "GND" (at 53.34 309.88 0)
     (effects (font (size 1.27 1.27)) (justify left bottom))
@@
     (effects (font (size 1.27 1.27)) (justify left bottom))
   )
+  (label "-U_TO_A_SPD_SAMPLE" (at 33.02 231.14 180)
+    (effects (font (size 1.27 1.27)) (justify right bottom))
+  )
   (label "-3V" (at 279.4 304.8 180)
     (effects (font (size 1.27 1.27)) (justify right bottom))
@@
     (effects (font (size 1.27 1.27)) (justify right bottom))
   )
+  (label "-A_TO_B_8-15_SPD_GATE" (at 45.72 111.76 0)
+    (effects (font (size 1.27 1.27)) (justify left bottom))
+  )
+  (label "-DC_SET_D_0-7" (at 45.72 193.04 0)
+    (effects (font (size 1.27 1.27)) (justify left bottom))
+  )
   (label "+3V" (at 751.84 297.18 0)
     (effects (font (size 1.27 1.27)) (justify left bottom))
@@
     (effects (font (size 1.27 1.27)) (justify right bottom))
   )
+  (label "-I_TO_B_SPD_GATE" (at 33.02 114.3 180)
+    (effects (font (size 1.27 1.27)) (justify right bottom))
+  )
   (label "GND" (at 751.84 195.58 0)
     (effects (font (size 1.27 1.27)) (justify left bottom))
@@
     (effects (font (size 1.27 1.27)) (justify left bottom))
   )
+  (label "+GATE_B_TO_D_0-7" (at 33.02 149.86 180)
+    (effects (font (size 1.27 1.27)) (justify right bottom))
+  )
   (label "+3V" (at 815.34 297.18 0)
     (effects (font (size 1.27 1.27)) (justify left bottom))
@@
     (effects (font (size 1.27 1.27)) (justify right bottom))
   )
+  (label "+GATE_I_TO_A_8-15" (at 45.72 109.22 0)
+    (effects (font (size 1.27 1.27)) (justify left bottom))
+  )
   (label "GND" (at 624.84 271.78 0)
     (effects (font (size 1.27 1.27)) (justify left bottom))
@@
     (effects (font (size 1.27 1.27)) (justify left bottom))
   )
-  (label "+3V" (at 53.34 220.98 0)
-    (effects (font (size 1.27 1.27)) (justify left bottom))
-  )
   (label "-EXCHANGE_A_AND_Q_SP_4-7" (at 363.22 193.04 0)
     (effects (font (size 1.27 1.27)) (justify left bottom))
@@
     (effects (font (size 1.27 1.27)) (justify left bottom))
   )
-  (label "+6V" (at 25.4 241.3 180)
-    (effects (font (size 1.27 1.27)) (justify right bottom))
-  )
   (label "-IO_BIT_15" (at 744.22 241.3 0)
     (effects (font (size 1.27 1.27)) (justify left bottom))
@@
     (effects (font (size 1.27 1.27)) (justify left bottom))
   )
+  (label "-A_TO_U_SPD_SAMPLE" (at 45.72 218.44 0)
+    (effects (font (size 1.27 1.27)) (justify left bottom))
+  )

Commit message: Finish page KM201-KM211
Connections:
- net +3V: no longer J355.b2 (Pin_b2), J356.b2 (Pin_b2)
- net +6V: no longer J355.a10 (Pin_a10), J356.a10 (Pin_a10)
- net +I1_POWERED: now also J362.a2 (Pin_a2), J362.b11 (Pin_b11), J362.b6 (Pin_b6)
- net +I2_CYCLE: now also J368.a2 (Pin_a2), J368.b10 (Pin_b10), J368.b6 (Pin_b6), J368.b9 (Pin_b9)
- net -3V: no longer J355.a5 (Pin_a5), J356.a5 (Pin_a5)
- net -I_O_ENTR_SAMPLE: now also J350.b5 (Pin_b5)
- net -I-O_BIT_5: now reaches J362.a6 (Pin_a6)
- net KM201_AL4: now reaches J362.a8 (Pin_a8)
- net KM201_AL4: now also J350.b8 (Pin_b8), J362.b12 (Pin_b12), J362.b4 (Pin_b4), J368.a12 (Pin_a12), J368.a8 (Pin_a8), J368.b12 (Pin_b12), J368.b5 (Pin_b5)
- net -I-O_BIT_8: now reaches J362.b3 (Pin_b3)
- net -I-O_BIT_1: now reaches J362.b9 (Pin_b9)
- net KM201_AC4: now reaches J368.a11 (Pin_a11)
- net KM201_AC4: now also J350.b10 (Pin_b10)
- net -I-O_BIT_15: now reaches J368.a6 (Pin_a6)
- net KM201_AD4: now reaches J368.a7 (Pin_a7)
- net KM201_AD4: now also J350.b11 (Pin_b11)
- net -I-O-BIT_14: now reaches J368.a9 (Pin_a9)
- net -I-O_BIT_13: now reaches J368.b3 (Pin_b3)
- net KM201_AS4: now reaches J368.b4 (Pin_b4)
- net KM201_AS4: now also J350.b9 (Pin_b9)
- net -I-O_BIT_12: now reaches J368.b8 (Pin_b8)
- net -CS_LEVEL_1: now reaches J356.a4 (Pin_a4)
- net -CS_LEVEL_1: now also J350.a4 (Pin_a4)
- net -PRINTER_C_S_REQ: now reaches J356.a6 (Pin_a6)
- net -PRINTER_C_S_REQ: now also J350.a5 (Pin_a5)
- net +CS_LEVEL_1: now reaches J356.a7 (Pin_a7)
- net +CS_LEVEL_1: now also J350.a6 (Pin_a6)
- net +CS_LEVEL_0: now reaches J355.b12 (Pin_b12)
- net +CS_LEVEL_0: now also J350.a10 (Pin_a10)
- net -CS_LEVELS: now reaches J350.a1 (Pin_a1)
Other:
- note added: "5800236"
- note added: "5800238"
- note added: "CABL 01A-A1N4"
- note added: "CABL 01A-C1N3"
