File: 1130_backplane/01B-B1.kicad_sch (KiCad schematic)
At the start: 86 parts

Commit message: Finish page KU101-KU111
Connections:
- net +D_REG_EQUAL_ZERO_CKT_2: now reaches J383.a7 (Pin_a7)
- net +D_REG_EQUAL_ZERO_CKT_2: now also J421.a11 (Pin_a11)
- net +D_REG_EQUAL_ZERO_CKT_1: now reaches J347.a3 (Pin_a3)
- net +D_REG_EQUAL_ZERO_CKT_1: now also J421.a2 (Pin_a2)
- net -A_REG_EQUAL_ZERO: now reaches J347.b3 (Pin_b3)
- net -A_REG_EQUAL_ZERO: now also J421.b1 (Pin_b1)
- net -I_BIT_10_OR_CCC_32_TO_ACC: now reaches J346.a10 (Pin_a10)
- net -I_BIT_12_OR_CCC_8_TO_ACC: now reaches J346.a11 (Pin_a11)
- net -I_BIT_14_CCC_4_CARRY_TO_ACC: now reaches J346.a12 (Pin_a12)
- net -I_BIT_11_OR_CCC_16_TO_ACC: now reaches J346.b10 (Pin_b10)
- net -I_BIT_13_OR_CCC_4_TO_ACC: now reaches J346.b11 (Pin_b11)
- net -I_BIT_15_CCC_1_OFLO_TO_ACC: now reaches J346.b12 (Pin_b12)
- net -A_BIT_0_OR_1: now reaches J421.a1 (Pin_a1)
- net -D_BIT_0_OR_1: now reaches J421.a3 (Pin_a3)
Other:
- note added: "DOT OR"

Commit message: Finish page KU201-KU211
Connections:
- net +CS_LVL_0_PWR: now reaches J350.a9 (Pin_a9)
Changed lines of the file:
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@@
     (effects (font (size 1.27 1.27)) (justify left bottom))
+  )
+  (label "+CS_LVL_0_PWR" (at 33.02 314.96 180)
+    (effects (font (size 1.27 1.27)) (justify right bottom))
   )
   (label "-GROUND_D08" (at 414.02 180.34 180)

Commit message: Finish page KU301-KU311, minor column label fix.
Connections:
- net -IX_ADDR_INHIBIT_SAR: now reaches J383.a11 (Pin_a11)
- net +IX_ADDR_INHIBIT_SAR: now reaches J383.b11 (Pin_b11)
- net -DC_RESET_B_0-7: now reaches J347.a1 (Pin_a1)
- net -DC_RESET_A_REG: now reaches J347.a7 (Pin_a7)
- net -DC_RESET_B_8-15: now reaches J345.b11 (Pin_b11)
- net -DC_RESET_IAR: now reaches J345.b12 (Pin_b12)
Changed lines of the file:
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@@
     (effects (font (size 1.27 1.27)) (justify left bottom))
   )
-  (text "H" (at 482.6 90.17 0)
+  (text "H" (at 481.33 90.17 0)
     (effects (font (size 5 5) (thickness 1) bold) (justify left bottom))
   )
@@
     (effects (font (size 1.27 1.27)) (justify left bottom))
   )
-  (text "H" (at 482.6 337.82 0)
+  (text "H" (at 481.33 337.82 0)
     (effects (font (size 5 5) (thickness 1) bold) (justify left bottom))
   )
@@
     (effects (font (size 1.27 1.27)) (justify right bottom))
   )
+  (label "-DC_RESET_B_0-7" (at 33.02 180.34 180)
+    (effects (font (size 1.27 1.27)) (justify right bottom))
+  )
   (label "+3V" (at 751.84 259.08 0)
     (effects (font (size 1.27 1.27)) (justify left bottom))
@@
     (effects (font (size 1.27 1.27)) (justify left bottom))
   )
+  (label "+IX_ADDR_INHIBIT_SAR" (at 412.75 50.8 90)
+    (effects (font (size 1.27 1.27)) (justify left bottom))
+  )
   (label "+3V" (at 307.34 259.08 0)
     (effects (font (size 1.27 1.27)) (justify left bottom))
@@
     (effects (font (size 1.27 1.27)) (justify left bottom))
   )
+  (label "-DC_RESET_B_8-15" (at 45.72 129.54 0)
+    (effects (font (size 1.27 1.27)) (justify left bottom))
+  )
   (label "GND" (at 688.34 309.88 0)
     (effects (font (size 1.27 1.27)) (justify left bottom))
@@
     (effects (font (size 1.27 1.27)) (justify right bottom))
   )
+  (label "-IX_ADDR_INHIBIT_SAR" (at 412.75 63.5 270)
+    (effects (font (size 1.27 1.27)) (justify right bottom))
+  )
   (label "+3V" (at 370.84 220.98 0)
     (effects (font (size 1.27 1.27)) (justify left bottom))
@@
     (effects (font (size 1.27 1.27)) (justify right bottom))
   )
+  (label "-DC_RESET_IAR" (at 45.72 132.08 0)
+    (effects (font (size 1.27 1.27)) (justify left bottom))
+  )
   (label "KM201_AD4" (at 45.72 320.04 0)
     (effects (font (size 1.27 1.27)) (justify left bottom))
@@
     (effects (font (size 1.27 1.27)) (justify left bottom))
   )
+  (label "-DC_RESET_A_REG" (at 33.02 195.58 180)
+    (effects (font (size 1.27 1.27)) (justify right bottom))
+  )
   (label "-3V" (at 88.9 114.3 180)

Commit message: Finish page MB101
Connections:
- net +IX_ADDR_INHIBIT_SAR: now also J385.b3 (Pin_b3)
- net -CS_LEVELS: now also J375.a2 (Pin_a2), J385.a11 (Pin_a11), J385.a3 (Pin_a3), J385.a6 (Pin_a6), J385.b12 (Pin_b12)
- net -IX_ADDR_INHIBIT_SAR: now also J385.a2 (Pin_a2), J385.b10 (Pin_b10)
- net +M_BIT_3: now reaches J375.a1 (Pin_a1)
- net +M_BIT_7: now reaches J375.a11 (Pin_a11)
- net +M_BIT_9: now reaches J375.a12 (Pin_a12)
- net +M_BIT_5: now reaches J375.a3 (Pin_a3)
- net +M_BIT_8: now reaches J375.a4 (Pin_a4)
- net MB101_AB4: now reaches J375.a6 (Pin_a6)
- net MB101_AB4: now also J385.a1 (Pin_a1)
- net +M_BIT_11: now reaches J375.a7 (Pin_a7)
- net +M_BIT_6: now reaches J375.a8 (Pin_a8)
- net +M_BIT_4: now reaches J375.a9 (Pin_a9)
- net -FILE_ADDR_3: now reaches J375.b1 (Pin_b1)
- net -FILE_ADDR_7: now reaches J375.b10 (Pin_b10)
- net +M_BIT_10: now reaches J375.b11 (Pin_b11)
- net -FILE_ADDR_9: now reaches J375.b12 (Pin_b12)
- net -FILE_ADDR_8: now reaches J375.b3 (Pin_b3)
- net -FILE_ADDR_4: now reaches J375.b4 (Pin_b4)
- net -FILE_ADDR_5: now reaches J375.b5 (Pin_b5)
- net -FILE_ADDR_11: now reaches J375.b6 (Pin_b6)
- net -FILE_ADDR_6: now reaches J375.b8 (Pin_b8)
- net -FILE_ADDR_10: now reaches J375.b9 (Pin_b9)
- net +M_BIT_15: now reaches J385.a12 (Pin_a12)
- net +M_BIT_13: now reaches J385.a4 (Pin_a4)
- net +M_BIT_12: now reaches J385.a7 (Pin_a7)
- net -DBL_WORD_ODD_ADDR: now reaches J385.a8 (Pin_a8)
- net -DPW_ODD_ADDR_SAR_15: now reaches J385.a9 (Pin_a9)
- net -DPW_ODD_ADDR_SAR_15: now also J385.b9 (Pin_b9)
- net -FILE_ADDR_13: now reaches J385.b1 (Pin_b1)
- net +M_BIT_14: now reaches J385.b11 (Pin_b11)
- net +M_ODD: now reaches J385.b4 (Pin_b4)
- net -FILE_ADDR_12: now reaches J385.b5 (Pin_b5)
- net -M_BIT_15: now reaches J385.b6 (Pin_b6)
Other:
- note added: "5800533"
- note added: "5803016"

Commit message: Actually finish MB101...
Connections:
- net +M_ODD: now also J419.b9 (Pin_b9)
- net -FILE_ADDR_10: now also J391.a10 (Pin_a10), J391.a7 (Pin_a7)
- net -FILE_ADDR_11: now also J391.b10 (Pin_b10)
- net -FILE_ADDR_12: now also J391.a11 (Pin_a11)
- net -FILE_ADDR_13: now also J391.b11 (Pin_b11)
- net -FILE_ADDR_3: now also J391.b1 (Pin_b1), J391.b2 (Pin_b2)
- net -FILE_ADDR_4: now also J391.a3 (Pin_a3)
- net -FILE_ADDR_5: now also J391.b3 (Pin_b3)
- net -FILE_ADDR_6: now also J391.a4 (Pin_a4)
- net -FILE_ADDR_7: now also J391.b4 (Pin_b4)
- net -FILE_ADDR_8: now also J391.a9 (Pin_a9)
- net -FILE_ADDR_9: now also J391.b9 (Pin_b9)
- net -FILE_ADDR_14: now reaches J383.a12 (Pin_a12)
- net -FILE_ADDR_14: now also J385.a9 (Pin_a9), J391.a12 (Pin_a12)
- net -FILE_ADDR_15: now reaches J383.b12 (Pin_b12)
- net -FILE_ADDR_15: now also J385.b9 (Pin_b9), J391.b12 (Pin_b12)
- removed net -DPW_ODD_ADDR_SAR_15: J385.a9 (Pin_a9), J385.b9 (Pin_b9)
Other:
- note added: "CABL 01B-C1T3"

Commit message: Finish page MB201
Connections:
- net +CS_LEVEL_0: now also J362.b8 (Pin_b8), J389.a12 (Pin_a12), J389.a3 (Pin_a3), J389.b12 (Pin_b12), J389.b4 (Pin_b4), J389.b6 (Pin_b6), J389.b8 (Pin_b8)
- net +CS_LEVEL_1: now also J368.b1 (Pin_b1)
- net +CS_LVL_0_PWR: now also J379.b11 (Pin_b11)
- net -FILE_ADDR_10: now also J368.a1 (Pin_a1), J379.b9 (Pin_b9)
- net -FILE_ADDR_11: now also J379.b6 (Pin_b6)
- net -FILE_ADDR_12: now also J389.b9 (Pin_b9)
- net -FILE_ADDR_13: now also J362.b5 (Pin_b5), J389.a6 (Pin_a6)
- net -FILE_ADDR_14: now also J389.a9 (Pin_a9), J389.b3 (Pin_b3)
- net -FILE_ADDR_15: now also J389.a1 (Pin_a1), J389.b5 (Pin_b5)
- net -FILE_ADDR_3: now also J379.b1 (Pin_b1)
- net -FILE_ADDR_4: now also J379.b4 (Pin_b4)
- net -FILE_ADDR_5: now also J379.b5 (Pin_b5)
- net -FILE_ADDR_6: now also J379.b8 (Pin_b8)
- net -FILE_ADDR_7: now also J379.b10 (Pin_b10)
- net -FILE_ADDR_8: now also J379.b3 (Pin_b3)
- net -FILE_ADDR_9: now also J379.b12 (Pin_b12)
- net +FILE_ADDR_BIT_14: now reaches J389.a2 (Pin_a2)
- net +FILE_ADDR_BIT_15: now reaches J389.a7 (Pin_a7)
- net +FILE_ADDR_BIT_13: now reaches J389.a8 (Pin_a8)
- net +PRINTER_ADDR_REG_1: now reaches J389.b1 (Pin_b1)
- net +PRINTER_ADDR_REG_1: now also J356.a1 (Pin_a1)
- net +PRINTER_ADDR_REG_2: now reaches J389.b10 (Pin_b10)
- net +PRINTER_ADDR_REG_2: now also J356.a2 (Pin_a2)
- net +FILE_ADDR_BIT_12: now reaches J389.b11 (Pin_b11)
- net +PRINTER_ADDR_REG_4: now reaches J362.a7 (Pin_a7)
- net +PRINTER_ADDR_REG_4: now also J356.a3 (Pin_a3)
- net +FILE_ADDR_BIT_4: now reaches J379.a1 (Pin_a1)
- net +FILE_ADDR_BIT_9: now reaches J379.a11 (Pin_a11)
- net +FILE_ADDR_BIT_3: now reaches J379.a2 (Pin_a2)
- net +FILE_ADDR_BIT_8: now reaches J379.a3 (Pin_a3)
- net +FILE_ADDR_BIT_6: now reaches J379.a4 (Pin_a4)
- net +FILE_ADDR_BIT_5: now reaches J379.a7 (Pin_a7)
- net +FILE_ADDR_BIT_7: now reaches J379.a8 (Pin_a8)
- net +FILE_ADDR_BIT_11: now reaches J379.a9 (Pin_a9)
Other:
- note added: "5803028"

Commit message: Finish page MC101
Connections:
- net +STORAGE_WRITE_CYCLE: now reaches J383.a1 (Pin_a1)
- net +STORAGE_WRITE_CYCLE: now also J383.a5 (Pin_a5), J391.a1 (Pin_a1), J391.a5 (Pin_a5)
- net +STORAGE_READ_CYCLE: now reaches J383.a6 (Pin_a6)
- net +STORAGE_READ_CYCLE: now also J391.a6 (Pin_a6)
- net +STORAGE_USE: now reaches J383.a8 (Pin_a8)
- net +STORAGE_USE: now also J391.a8 (Pin_a8)
- net +STORAGE_SELECT: now reaches J383.b8 (Pin_b8)
- net +STORAGE_SELECT: now also J391.b8 (Pin_b8)
Changed lines of the file:
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@@
     (effects (font (size 1.27 1.27)) (justify left bottom))
+  )
+  (label "+STORAGE_READ_CYCLE" (at 438.15 63.5 270)
+    (effects (font (size 1.27 1.27)) (justify right bottom))
   )
   (label "GND" (at 434.34 309.88 0)
@@
     (effects (font (size 1.27 1.27)) (justify left bottom))
   )
+  (label "+STORAGE_WRITE_CYCLE" (at 387.35 63.5 270)
+    (effects (font (size 1.27 1.27)) (justify right bottom))
+  )
   (label "-3V" (at 469.9 190.5 180)
     (effects (font (size 1.27 1.27)) (justify right bottom))
@@
     (effects (font (size 1.27 1.27)) (justify left bottom))
   )
+  (label "+STORAGE_SELECT" (at 405.13 50.8 90)
+    (effects (font (size 1.27 1.27)) (justify left bottom))
+  )
   (label "-FILE_ADDR_5" (at 265.43 31.75 0)
     (effects (font (size 1.27 1.27)) (justify left bottom))
@@
     (effects (font (size 1.27 1.27)) (justify left bottom))
   )
+  (label "+STORAGE_WRITE_CYCLE" (at 397.51 63.5 270)
+    (effects (font (size 1.27 1.27)) (justify right bottom))
+  )
   (label "-EXCHG_A_AND_Q_SPD_SAMPLE" (at 350.52 185.42 180)
     (effects (font (size 1.27 1.27)) (justify right bottom))
@@
     (effects (font (size 1.27 1.27)) (justify left bottom))
   )
+  (label "+STORAGE_USE" (at 443.23 63.5 270)
+    (effects (font (size 1.27 1.27)) (justify right bottom))
+  )
   (label "+EVEN_PARITY_1" (at 45.72 187.96 0)
     (effects (font (size 1.27 1.27)) (justify left bottom))
@@
     (effects (font (size 1.27 1.27)) (justify right bottom))
   )
+  (label "+STORAGE_WRITE_CYCLE" (at 425.45 63.5 270)
+    (effects (font (size 1.27 1.27)) (justify right bottom))
+  )
   (label "-AND_SP" (at 350.52 220.98 180)
     (effects (font (size 1.27 1.27)) (justify right bottom))
@@
     (effects (font (size 1.27 1.27)) (justify right bottom))
   )
+  (label "+STORAGE_SELECT" (at 443.23 50.8 90)
+    (effects (font (size 1.27 1.27)) (justify left bottom))
+  )
   (label "GND" (at 116.84 119.38 0)
     (effects (font (size 1.27 1.27)) (justify left bottom))
@@
     (effects (font (size 1.27 1.27)) (justify right bottom))
   )
+  (label "+STORAGE_READ_CYCLE" (at 400.05 63.5 270)
+    (effects (font (size 1.27 1.27)) (justify right bottom))
+  )
   (label "MB101_AQ4" (at 363.22 127 0)
     (effects (font (size 1.27 1.27)) (justify left bottom))
@@
     (effects (font (size 1.27 1.27)) (justify left bottom))
   )
+  (label "+STORAGE_USE" (at 405.13 63.5 270)
+    (effects (font (size 1.27 1.27)) (justify right bottom))
+  )
   (label "-A_TO_M_SP_8-15" (at 426.72 147.32 0)
     (effects (font (size 1.27 1.27)) (justify left bottom))
@@
     (effects (font (size 1.27 1.27)) (justify right bottom))
   )
+  (label "+STORAGE_WRITE_CYCLE" (at 435.61 63.5 270)
+    (effects (font (size 1.27 1.27)) (justify right bottom))
+  )

Commit message: Finish page RA101-RA171
Connections:
- net +ACC_BIT_0_SHIFT_RT_ENTRY: now also J353.a12 (Pin_a12)
- net -ACC_BIT_0_SHIFT_RT_ENTRY: now also J353.b12 (Pin_b12)
- net -ADD_SUB_EOR_GATE: now also J354.b6 (Pin_b6), J360.b6 (Pin_b6), J366.b6 (Pin_b6), J372.b6 (Pin_b6)
- net -ADD_SUB_OR_EOR_GATE: now also J353.a9 (Pin_a9), J359.a9 (Pin_a9), J365.a9 (Pin_a9), J371.a9 (Pin_a9)
- net -AND_SP: now also J354.b3 (Pin_b3), J360.b3 (Pin_b3), J366.b3 (Pin_b3), J372.b3 (Pin_b3)
- net -A_BIT_0_OR_1: now also J354.a8 (Pin_a8), J360.a8 (Pin_a8), J366.a8 (Pin_a8), J372.a8 (Pin_a8)
- net -A_TO_U_SP_0-7: now also J353.a3 (Pin_a3), J359.a3 (Pin_a3), J365.a3 (Pin_a3), J371.a3 (Pin_a3)
- net -DC_RESET_A_REG: now also J353.a8 (Pin_a8), J359.a8 (Pin_a8), J365.a8 (Pin_a8), J371.a8 (Pin_a8)
- net -EXCHANGE_A_AND_Q_SP_0-3: now also J353.b3 (Pin_b3), J359.b3 (Pin_b3)
- net -EXCHANGE_A_AND_Q_SP_4-7: now also J365.b3 (Pin_b3), J371.b3 (Pin_b3)
- net -SHIFT_LEFT_A_SP_0-7: now also J354.a7 (Pin_a7), J360.a7 (Pin_a7), J366.a7 (Pin_a7), J372.a7 (Pin_a7)
- net -SHIFT_RIGHT_A_SP_0-7: now also J354.b1 (Pin_b1), J360.b1 (Pin_b1), J366.b1 (Pin_b1), J372.b1 (Pin_b1)
- net -U_TO_A_SP_0-7: now also J354.a2 (Pin_a2), J360.a2 (Pin_a2), J366.a2 (Pin_a2), J372.a2 (Pin_a2)
- net GND: now also J354.a1 (Pin_a1), J360.a1 (Pin_a1), J366.a1 (Pin_a1), J372.a1 (Pin_a1)
- net +A_BIT_2: now reaches J419.a11 (Pin_a11)
- net +A_BIT_2: now also J354.a9 (Pin_a9), J359.b10 (Pin_b10)
- net +A_BIT_0: now reaches J419.a9 (Pin_a9)
- net +A_BIT_0: now also J348.a5 (Pin_a5), J353.b10 (Pin_b10)
- net +A_BIT_1: now reaches J419.b10 (Pin_b10)
- net +A_BIT_1: now also J354.b4 (Pin_b4), J359.a12 (Pin_a12)
- net +A_BIT_3: now reaches J419.b11 (Pin_b11)
- net +A_BIT_3: now also J360.b4 (Pin_b4), J365.a12 (Pin_a12)
- net -U_BIT_2: now reaches J359.a1 (Pin_a1)
- net -U_BIT_2: now also J355.a2 (Pin_a2)
- net -I_BIT_2_TO_ACC: now reaches J359.a11 (Pin_a11)
- net +Q_BIT_2: now reaches J359.a4 (Pin_a4)
- net +Q_BIT_3: now reaches J359.a6 (Pin_a6)
- net -A_BIT_2: now reaches J359.a7 (Pin_a7)
- net -A_BIT_2: now also J354.b8 (Pin_b8)
- net +D_BIT_2: now reaches J359.b11 (Pin_b11)
- net -A_BIT_1: now reaches J359.b12 (Pin_b12)
- net -A_BIT_1: now also J348.b6 (Pin_b6), J354.a4 (Pin_a4)
- net -U_BIT_3: now reaches J359.b5 (Pin_b5)
- net -U_BIT_3: now also J355.b3 (Pin_b3)
- net -U_BIT_4: now reaches J365.a1 (Pin_a1)
- net -U_BIT_4: now also J355.a3 (Pin_a3)
- net -I_BIT_4_TO_ACC: now reaches J365.a11 (Pin_a11)
- net +Q_BIT_4: now reaches J365.a4 (Pin_a4)
- net +Q_BIT_5: now reaches J365.a6 (Pin_a6)
- net -A_BIT_4: now reaches J365.a7 (Pin_a7)
- net -A_BIT_4: now also J360.b8 (Pin_b8)
- net +A_BIT_4: now reaches J365.b10 (Pin_b10)
- net +A_BIT_4: now also J360.a9 (Pin_a9), J425.a9 (Pin_a9)
- net +D_BIT_4: now reaches J365.b11 (Pin_b11)
- net -A_BIT_3: now reaches J365.b12 (Pin_b12)
- net -A_BIT_3: now also J360.a4 (Pin_a4)
- net -U_BIT_5: now reaches J365.b5 (Pin_b5)
- net -U_BIT_5: now also J348.a12 (Pin_a12), J355.b4 (Pin_b4)
- net -U_BIT_0: now reaches J353.a1 (Pin_a1)
- net -U_BIT_0: now also J348.a9 (Pin_a9), J355.a1 (Pin_a1)
- net -I_BIT_0_TO_ACC: now reaches J353.a11 (Pin_a11)
- net +Q_BIT_0: now reaches J353.a4 (Pin_a4)
- net +Q_BIT_1: now reaches J353.a6 (Pin_a6)
- net -A_BIT_0: now reaches J353.a7 (Pin_a7)
- net -D_BIT_0: now reaches J353.b11 (Pin_b11)
- net -U_BIT_1: now reaches J353.b5 (Pin_b5)
- net -U_BIT_1: now also J355.b1 (Pin_b1)
- net -U_BIT_7: now reaches J348.b12 (Pin_b12)
- net -U_BIT_7: now also J355.b5 (Pin_b5), J371.b5 (Pin_b5)
- net +A_BIT_6: now reaches J425.a11 (Pin_a11)
- net +A_BIT_6: now also J366.a9 (Pin_a9), J371.b10 (Pin_b10)
- net +A_BIT_5: now reaches J425.b10 (Pin_b10)
- net +A_BIT_5: now also J366.b4 (Pin_b4), J371.a12 (Pin_a12)
- net +A_BIT_7: now reaches J425.b11 (Pin_b11)
- net +A_BIT_7: now also J372.b4 (Pin_b4)
- net -U_BIT_6: now reaches J371.a1 (Pin_a1)
- net -U_BIT_6: now also J355.a4 (Pin_a4)
- net -I_BIT_6_TO_ACC: now reaches J371.a11 (Pin_a11)
- net +Q_BIT_6: now reaches J371.a4 (Pin_a4)
- net +Q_BIT_7: now reaches J371.a6 (Pin_a6)
- net -A_BIT_6: now reaches J371.a7 (Pin_a7)
- net -A_BIT_6: now also J366.b8 (Pin_b8)
- net +D_BIT_6: now reaches J371.b11 (Pin_b11)
- net -A_BIT_5: now reaches J371.b12 (Pin_b12)
- net -A_BIT_5: now also J366.a4 (Pin_a4)
- net -I_BIT_1_TO_ACC: now reaches J354.a3 (Pin_a3)
- net +D_BIT_1: now reaches J354.b5 (Pin_b5)
- net -I_BIT_5_TO_ACC: now reaches J366.a3 (Pin_a3)
- net +D_BIT_5: now reaches J366.b5 (Pin_b5)
- net -I_BIT_7_TO_ACC: now reaches J372.a3 (Pin_a3)
- net -A_BIT_7: now reaches J372.a4 (Pin_a4)
- net +A_BIT_8: now reaches J372.a9 (Pin_a9)
- net +D_BIT_7: now reaches J372.b5 (Pin_b5)
- net -A_BIT_8: now reaches J372.b8 (Pin_b8)
- net -I_BIT_3_TO_ACC: now reaches J360.a3 (Pin_a3)
- net +D_BIT_3: now reaches J360.b5 (Pin_b5)
Other:
- note added: "5804617"
