File: 1130_backplane/01A-C1.kicad_sch (KiCad schematic)
At the start: 86 parts

Commit message: Finish page KM201-KM211
Connections:
- net +3V: no longer J254.b2 (Pin_b2)
- net +6V: no longer J254.a10 (Pin_a10)
- net -3V: no longer J254.a5 (Pin_a5)
- net -CS_LEVEL_0: now reaches J257.a1 (Pin_a1)
- net +CS_LEVEL_0: now reaches J254.b12 (Pin_b12)
Other:
- note added: "CABL 01B-B1B6"
Changed lines of the file:
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@@
     (stroke (width 0) (type default) (color 0 0 0 0))
   )
-  (wire (pts (xy 807.72 144.78) (xy 815.34 144.78))
-    (stroke (width 0) (type default) (color 0 0 0 0))
-  )
   (polyline (pts (xy 322.58 369.57) (xy 323.85 369.57))
     (stroke (width 0) (type solid) (color 0 0 0 0))
@@
     (stroke (width 0) (type default) (color 0 0 0 0))
   )
-  (wire (pts (xy 787.4 165.1) (xy 795.02 165.1))
-    (stroke (width 0) (type default) (color 0 0 0 0))
-  )
   (polyline (pts (xy 29.21 71.12) (xy 30.48 71.12))
     (stroke (width 0) (type solid) (color 0 0 0 0))
@@
     (stroke (width 0) (type solid) (color 0 0 0 0))
   )
-  (wire (pts (xy 787.4 152.4) (xy 795.02 152.4))
-    (stroke (width 0) (type default) (color 0 0 0 0))
-  )
   (wire (pts (xy 744.22 220.98) (xy 751.84 220.98))
     (stroke (width 0) (type default) (color 0 0 0 0))
@@
     (effects (font (size 5 5) (thickness 1) bold) (justify left bottom))
   )
+  (text "CABL 01B-B1B6" (at 793.75 139.7 0)
+    (effects (font (size 1.27 1.27)) (justify left bottom))
+  )
   (text "3" (at 833.12 160.02 0)
     (effects (font (size 5 5) (thickness 1) bold) (justify left bottom))
@@
     (effects (font (size 1.27 1.27)) (justify left bottom))
   )
-  (label "+6V" (at 787.4 165.1 180)
-    (effects (font (size 1.27 1.27)) (justify right bottom))
-  )
   (label "GND" (at 624.84 233.68 0)
     (effects (font (size 1.27 1.27)) (justify left bottom))
@@
     (effects (font (size 1.27 1.27)) (justify right bottom))
   )
+  (label "-CS_LEVEL_0" (at 795.02 256.54 180)
+    (effects (font (size 1.27 1.27)) (justify right bottom))
+  )
   (label "+3V" (at 307.34 297.18 0)
     (effects (font (size 1.27 1.27)) (justify left bottom))
@@
     (effects (font (size 1.27 1.27)) (justify left bottom))
   )
-  (label "-3V" (at 787.4 152.4 180)
-    (effects (font (size 1.27 1.27)) (justify right bottom))
-  )
   (label "GND" (at 751.84 157.48 0)
     (effects (font (size 1.27 1.27)) (justify left bottom))
@@
     (effects (font (size 1.27 1.27)) (justify right bottom))
   )
-  (label "+3V" (at 815.34 144.78 0)
-    (effects (font (size 1.27 1.27)) (justify left bottom))
-  )
   (label "+3V" (at 434.34 220.98 0)
     (effects (font (size 1.27 1.27)) (justify left bottom))
@@
     (effects (font (size 1.27 1.27)) (justify left bottom))
   )
+  (label "+CS_LEVEL_0" (at 807.72 170.18 0)
+    (effects (font (size 1.27 1.27)) (justify left bottom))
+  )

Commit message: Finish page KM301-KM321
Connections:
- net -INTERRUPT_LEVEL_4: now reaches J257.a8 (Pin_a8)
- net -INTERRUPT_LEVEL_4: now also J212.b6 (Pin_b6)
- net +PRINTER_LVL_1_INTERRUPT_REQ: now reaches J211.a12 (Pin_a12)
- net +PRINTER_LVL_1_INTERRUPT_REQ: now also J255.b10 (Pin_b10)
Changed lines of the file:
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@@
+    (effects (font (size 1.27 1.27)) (justify right bottom))
+  )
+  (label "-INTERRUPT_LEVEL_4" (at 795.02 274.32 180)
     (effects (font (size 1.27 1.27)) (justify right bottom))
   )
@@
     (effects (font (size 1.27 1.27)) (justify right bottom))
   )
+  (label "-INTERRUPT_LEVEL_4" (at 400.05 356.87 90)
+    (effects (font (size 1.27 1.27)) (justify left bottom))
+  )
   (label "+AREA_6" (at 412.75 63.5 270)
     (effects (font (size 1.27 1.27)) (justify right bottom))
@@
     (effects (font (size 1.27 1.27)) (justify left bottom))
   )
+  (label "+PRINTER_LVL_1_INTERRUPT_REQ" (at 807.72 203.2 0)
+    (effects (font (size 1.27 1.27)) (justify left bottom))
+  )
   (label "-3V" (at 723.9 266.7 180)
     (effects (font (size 1.27 1.27)) (justify right bottom))
@@
     (effects (font (size 1.27 1.27)) (justify right bottom))
   )
+  (label "+PRINTER_LVL_1_INTERRUPT_REQ" (at 415.29 63.5 270)
+    (effects (font (size 1.27 1.27)) (justify right bottom))
+  )

Commit message: Finish page KR101-KR111
Connections:
- net KR111_AY6: now reaches J257.b1 (Pin_b1)
- net KR111_AY6: now also J194.b8 (Pin_b8)
- net -PARITY_STOP: now reaches J257.b10 (Pin_b10)
- net -PARITY_STOP: now also J178.b10 (Pin_b10)
- net -PARITY_CHECK_LAMP_DR: now reaches J176.b11 (Pin_b11)
- net -PARITY_CHECK_LAMP_DR: now also J194.a8 (Pin_a8)
- net +48_VOLTS: now reaches J194.a4 (Pin_a4)
Other:
- note added: "5803819"
- note added: "CABL 01A-B1N7"
Changed lines of the file:
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@@
+    (effects (font (size 1.27 1.27)) (justify left bottom))
+  )
+  (text "CABL 01A-B1N7" (at 31.75 292.1 0)
     (effects (font (size 1.27 1.27)) (justify left bottom))
   )
@@
     (effects (font (size 5 5) (thickness 1) bold) (justify left bottom))
   )
+  (text "5803819" (at 226.06 215.9 0)
+    (effects (font (size 1.27 1.27)) (justify left bottom))
+  )
   (text "D" (at 311.15 368.3 0)
     (effects (font (size 1.27 1.27)) (justify left bottom))
@@
     (effects (font (size 1.27 1.27)) (justify right bottom))
   )
+  (label "-PARITY_CHECK_LAMP_DR" (at 223.52 236.22 180)
+    (effects (font (size 1.27 1.27)) (justify right bottom))
+  )
   (label "+6V" (at 660.4 241.3 180)
     (effects (font (size 1.27 1.27)) (justify right bottom))
@@
     (effects (font (size 1.27 1.27)) (justify right bottom))
   )
+  (label "KR111_AY6" (at 807.72 256.54 0)
+    (effects (font (size 1.27 1.27)) (justify left bottom))
+  )
   (label "+AREA_8" (at 392.43 356.87 90)
     (effects (font (size 1.27 1.27)) (justify left bottom))
@@
     (effects (font (size 1.27 1.27)) (justify left bottom))
   )
+  (label "KR111_AY6" (at 236.22 236.22 0)
+    (effects (font (size 1.27 1.27)) (justify left bottom))
+  )
   (label "+6V" (at 469.9 317.5 180)
     (effects (font (size 1.27 1.27)) (justify right bottom))
@@
     (effects (font (size 1.27 1.27)) (justify left bottom))
   )
+  (label "+48_VOLTS" (at 223.52 226.06 180)
+    (effects (font (size 1.27 1.27)) (justify right bottom))
+  )
   (label "-3V" (at 88.9 266.7 180)
     (effects (font (size 1.27 1.27)) (justify right bottom))
@@
     (effects (font (size 1.27 1.27)) (justify left bottom))
   )
+  (label "-PARITY_CHECK_LAMP_DR" (at 45.72 243.84 0)
+    (effects (font (size 1.27 1.27)) (justify left bottom))
+  )
   (label "+3V" (at 688.34 182.88 0)
     (effects (font (size 1.27 1.27)) (justify left bottom))
@@
     (effects (font (size 1.27 1.27)) (justify left bottom))
   )
+  (label "-PARITY_STOP" (at 45.72 317.5 0)
+    (effects (font (size 1.27 1.27)) (justify left bottom))
+  )
   (label "+AREA_2" (at 350.52 129.54 180)
     (effects (font (size 1.27 1.27)) (justify right bottom))
@@
     (effects (font (size 1.27 1.27)) (justify right bottom))
   )
+  (label "-PARITY_STOP" (at 807.72 279.4 0)
+    (effects (font (size 1.27 1.27)) (justify left bottom))
+  )
   (label "-3V" (at 469.9 228.6 180)

Commit message: Finish page KT301-KT331
Connections:
- net -PROG_START_KEY_1: now reaches J257.a3 (Pin_a3)
- net -PROG_START_KEY_1: now also J178.a3 (Pin_a3)
- net -CE_KEY_SW: now reaches J257.b9 (Pin_b9)
- net +POWER_ON_RESET: now reaches J255.b4 (Pin_b4)
- net +POWER_ON_RESET: now also J178.a8 (Pin_a8)
Changed lines of the file:
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@@
     (effects (font (size 1.27 1.27)) (justify right bottom))
+  )
+  (label "-CE_KEY_SW" (at 807.72 276.86 0)
+    (effects (font (size 1.27 1.27)) (justify left bottom))
   )
   (label "KR111_AY6" (at 807.72 256.54 0)
@@
     (effects (font (size 1.27 1.27)) (justify right bottom))
   )
+  (label "-PROG_START_KEY_1" (at 33.02 299.72 180)
+    (effects (font (size 1.27 1.27)) (justify right bottom))
+  )
   (label "GND" (at 440.69 43.18 90)
     (effects (font (size 1.27 1.27)) (justify left bottom))
@@
     (effects (font (size 1.27 1.27)) (justify right bottom))
   )
+  (label "-PROG_START_KEY_1" (at 795.02 261.62 180)
+    (effects (font (size 1.27 1.27)) (justify right bottom))
+  )
   (label "-3V" (at 279.4 190.5 180)
     (effects (font (size 1.27 1.27)) (justify right bottom))
@@
     (effects (font (size 1.27 1.27)) (justify right bottom))
   )
+  (label "+POWER_ON_RESET" (at 807.72 187.96 0)
+    (effects (font (size 1.27 1.27)) (justify left bottom))
+  )
   (label "DU111_AK4" (at 223.52 170.18 180)
     (effects (font (size 1.27 1.27)) (justify right bottom))
@@
     (effects (font (size 1.27 1.27)) (justify left bottom))
   )
+  (label "+POWER_ON_RESET" (at 33.02 312.42 180)
+    (effects (font (size 1.27 1.27)) (justify right bottom))
+  )
   (label "-IO_BIT_10" (at 795.02 119.38 180)

Commit message: Finish page KU201-KU211
Connections:
- net +3V: no longer J177.b2 (Pin_b2)
- net +6V: no longer J177.a10 (Pin_a10)
- net -3V: no longer J177.a5 (Pin_a5)
- net +CPU_STOP_LATCH: now reaches J257.b8 (Pin_b8)
- net +CPU_STOP_LATCH: now also J178.b9 (Pin_b9)
- net +T6_PWR_1: now reaches J177.a11 (Pin_a11)
- net +T6_PWR_1: now also J255.a11 (Pin_a11)
- net +T4_PWR: now reaches J177.a12 (Pin_a12)
- net +T4_PWR: now also J255.a12 (Pin_a12)
- net +X4_PWR: now reaches J177.b11 (Pin_b11)
- net +X4_PWR: now also J255.b11 (Pin_b11)
- net -X6_PWR: now reaches J177.b12 (Pin_b12)
- net -X6_PWR: now also J255.b12 (Pin_b12)
- net +OSC_A_PWR: now reaches J255.b9 (Pin_b9)
- net +OSC_A_PWR: now also J177.a10 (Pin_a10)
Other:
- note added: "CABL 01A-B1N6"
Changed lines of the file:
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@@
     (stroke (width 0) (type solid) (color 0 0 0 0))
-  )
-  (wire (pts (xy 25.4 266.7) (xy 33.02 266.7))
-    (stroke (width 0) (type default) (color 0 0 0 0))
   )
   (wire (pts (xy 744.22 106.68) (xy 751.84 106.68))
@@
     (stroke (width 0) (type solid) (color 0 0 0 0))
   )
-  (wire (pts (xy 45.72 259.08) (xy 53.34 259.08))
-    (stroke (width 0) (type default) (color 0 0 0 0))
-  )
   (polyline (pts (xy 312.42 370.84) (xy 312.42 369.57))
     (stroke (width 0) (type solid) (color 0 0 0 0))
@@
     (stroke (width 0) (type default) (color 0 0 0 0))
   )
-  (wire (pts (xy 25.4 279.4) (xy 33.02 279.4))
-    (stroke (width 0) (type default) (color 0 0 0 0))
-  )
   (polyline (pts (xy 29.21 63.5) (xy 30.48 63.5))
     (stroke (width 0) (type solid) (color 0 0 0 0))
@@
     (effects (font (size 1.27 1.27)) (justify left bottom))
   )
+  (text "CABL 01A-B1N6" (at 31.75 254 0)
+    (effects (font (size 1.27 1.27)) (justify left bottom))
+  )
   (text "6" (at 21.59 53.34 0)
     (effects (font (size 1.27 1.27)) (justify left bottom))
@@
     (effects (font (size 1.27 1.27)) (justify left bottom))
   )
+  (label "+OSC_A_PWR" (at 807.72 200.66 0)
+    (effects (font (size 1.27 1.27)) (justify left bottom))
+  )
   (label "-XIO_TIME_GATE" (at 426.72 193.04 0)
     (effects (font (size 1.27 1.27)) (justify left bottom))
@@
     (effects (font (size 1.27 1.27)) (justify left bottom))
   )
+  (label "+T4_PWR" (at 795.02 208.28 180)
+    (effects (font (size 1.27 1.27)) (justify right bottom))
+  )
   (label "+3V" (at 497.84 220.98 0)
     (effects (font (size 1.27 1.27)) (justify left bottom))
@@
     (effects (font (size 1.27 1.27)) (justify left bottom))
   )
+  (label "+T6_PWR_1" (at 795.02 205.74 180)
+    (effects (font (size 1.27 1.27)) (justify right bottom))
+  )
   (label "DU101_AD4" (at 426.72 170.18 0)
     (effects (font (size 1.27 1.27)) (justify left bottom))
@@
     (effects (font (size 1.27 1.27)) (justify left bottom))
   )
+  (label "+T4_PWR" (at 33.02 284.48 180)
+    (effects (font (size 1.27 1.27)) (justify right bottom))
+  )
   (label "GND" (at 751.84 195.58 0)
     (effects (font (size 1.27 1.27)) (justify left bottom))
@@
     (effects (font (size 1.27 1.27)) (justify right bottom))
   )
-  (label "+6V" (at 25.4 279.4 180)
-    (effects (font (size 1.27 1.27)) (justify right bottom))
-  )
   (label "-3V" (at 533.4 228.6 180)
     (effects (font (size 1.27 1.27)) (justify right bottom))
@@
     (effects (font (size 1.27 1.27)) (justify left bottom))
   )
-  (label "+3V" (at 53.34 259.08 0)
-    (effects (font (size 1.27 1.27)) (justify left bottom))
-  )
   (label "+6V" (at 596.9 241.3 180)
     (effects (font (size 1.27 1.27)) (justify right bottom))
@@
     (effects (font (size 1.27 1.27)) (justify left bottom))
   )
+  (label "+CPU_STOP_LATCH" (at 807.72 274.32 0)
+    (effects (font (size 1.27 1.27)) (justify left bottom))
+  )
   (label "-3V" (at 279.4 304.8 180)
     (effects (font (size 1.27 1.27)) (justify right bottom))
@@
     (effects (font (size 1.27 1.27)) (justify left bottom))
   )
+  (label "+X4_PWR" (at 45.72 281.94 0)
+    (effects (font (size 1.27 1.27)) (justify left bottom))
+  )
   (label "-IO_BIT_13" (at 367.03 50.8 90)
     (effects (font (size 1.27 1.27)) (justify left bottom))
@@
     (effects (font (size 1.27 1.27)) (justify left bottom))
   )
+  (label "+OSC_A_PWR" (at 33.02 279.4 180)
+    (effects (font (size 1.27 1.27)) (justify right bottom))
+  )
   (label "GND" (at 751.84 119.38 0)
     (effects (font (size 1.27 1.27)) (justify left bottom))
@@
     (effects (font (size 1.27 1.27)) (justify right bottom))
   )
+  (label "+X4_PWR" (at 807.72 205.74 0)
+    (effects (font (size 1.27 1.27)) (justify left bottom))
+  )
   (label "GND" (at 478.79 43.18 90)
     (effects (font (size 1.27 1.27)) (justify left bottom))
@@
     (effects (font (size 1.27 1.27)) (justify right bottom))
   )
+  (label "-X6_PWR" (at 807.72 208.28 0)
+    (effects (font (size 1.27 1.27)) (justify left bottom))
+  )
   (label "-XIO_SENSE_RESET_15" (at 363.22 124.46 0)
     (effects (font (size 1.27 1.27)) (justify left bottom))
@@
     (effects (font (size 1.27 1.27)) (justify right bottom))
   )
+  (label "-X6_PWR" (at 45.72 284.48 0)
+    (effects (font (size 1.27 1.27)) (justify left bottom))
+  )
   (label "+3V" (at 561.34 259.08 0)
     (effects (font (size 1.27 1.27)) (justify left bottom))
@@
     (effects (font (size 1.27 1.27)) (justify left bottom))
   )
+  (label "+T6_PWR_1" (at 33.02 281.94 180)
+    (effects (font (size 1.27 1.27)) (justify right bottom))
+  )
   (label "-3V" (at 152.4 152.4 180)
     (effects (font (size 1.27 1.27)) (justify right bottom))
@@
     (effects (font (size 1.27 1.27)) (justify left bottom))
   )
-  (label "-3V" (at 25.4 266.7 180)
-    (effects (font (size 1.27 1.27)) (justify right bottom))
-  )
   (label "+PHASE_B" (at 45.72 320.04 0)
     (effects (font (size 1.27 1.27)) (justify left bottom))
   )
+  (label "+CPU_STOP_LATCH" (at 45.72 314.96 0)
+    (effects (font (size 1.27 1.27)) (justify left bottom))
+  )

Commit message: Finish page KU301-KU311, minor column label fix.
Connections:
- net -DC_RESET_IAR: now reaches J257.b3 (Pin_b3)
- net -DC_RESET_IAR: now also J178.b2 (Pin_b2)
Changed lines of the file:
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@@
     (effects (font (size 5 5) (thickness 1) bold) (justify left bottom))
   )
-  (text "H" (at 482.6 337.82 0)
+  (text "H" (at 481.33 337.82 0)
     (effects (font (size 5 5) (thickness 1) bold) (justify left bottom))
   )
@@
     (effects (font (size 1.27 1.27)) (justify left bottom))
   )
-  (text "H" (at 482.6 90.17 0)
+  (text "H" (at 481.33 90.17 0)
     (effects (font (size 5 5) (thickness 1) bold) (justify left bottom))
   )
@@
     (effects (font (size 1.27 1.27)) (justify right bottom))
   )
+  (label "-DC_RESET_IAR" (at 45.72 297.18 0)
+    (effects (font (size 1.27 1.27)) (justify left bottom))
+  )
   (label "+6V" (at 152.4 279.4 180)
     (effects (font (size 1.27 1.27)) (justify right bottom))
@@
     (effects (font (size 1.27 1.27)) (justify right bottom))
   )
+  (label "-DC_RESET_IAR" (at 807.72 261.62 0)
+    (effects (font (size 1.27 1.27)) (justify left bottom))
+  )
   (label "-IO_BIT_13" (at 807.72 124.46 0)

Commit message: Finish page KW101. Add 48V bus for 01A-C1
Connections:
- net +OSC_A_PWR: now also J218.b4 (Pin_b4)
- net +RUN_PROG_LOAD_DOT_ON_RUN: now also J218.b3 (Pin_b3)
- net -CE_KEY_SW: now also J218.b8 (Pin_b8)
- net -X6_PWR: now also J218.b12 (Pin_b12)
- net -METER_RUN: now reaches J176.a12 (Pin_a12)
- net -METER_RUN: now also J218.a1 (Pin_a1)
- net -RUN_LAMP_DR: now reaches J176.b8 (Pin_b8)
- net -RUN_LAMP_DR: now also J194.a7 (Pin_a7), J208.a2 (Pin_a2)
- net +CPU_RUN: now reaches J178.b6 (Pin_b6)
- net +CPU_RUN: now also J208.b3 (Pin_b3)
- net KW101_AB4: now reaches J218.a2 (Pin_a2)
- net KW101_AB4: now also J218.b10 (Pin_b10)
- net KW101_AN4: now reaches J218.a3 (Pin_a3)
- net KW101_AN4: now also J218.a6 (Pin_a6)
- net -ACCESS_DRIVE: now reaches J218.b11 (Pin_b11)
- net +48_VOLTS renamed +48V
Changed lines of the file:
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@@
     (stroke (width 0) (type solid) (color 0 0 0 0))
+  )
+  (wire (pts (xy 210.82 226.06) (xy 223.52 226.06))
+    (stroke (width 0) (type default) (color 0 0 0 0))
   )
   (polyline (pts (xy 34.29 44.45) (xy 34.29 45.72))
@@
     (effects (font (size 5 5) (thickness 1) bold) (justify left bottom))
   )
+  (text "5803819" (at 416.56 292.1 0)
+    (effects (font (size 1.27 1.27)) (justify left bottom))
+  )
   (text "E" (at 299.72 379.73 0)
     (effects (font (size 1.27 1.27)) (justify left bottom))
@@
     (effects (font (size 5 5) (thickness 1) bold) (justify left bottom))
   )
+  (text "5800000" (at 353.06 292.1 0)
+    (effects (font (size 1.27 1.27)) (justify left bottom))
+  )
   (text "5" (at 833.12 236.22 0)
     (effects (font (size 5 5) (thickness 1) bold) (justify left bottom))
@@
     (effects (font (size 1.27 1.27)) (justify left bottom))
   )
+  (label "KW101_AB4" (at 414.02 297.18 180)
+    (effects (font (size 1.27 1.27)) (justify right bottom))
+  )
   (label "+AREA_4" (at 350.52 147.32 180)
     (effects (font (size 1.27 1.27)) (justify right bottom))
@@
     (effects (font (size 1.27 1.27)) (justify left bottom))
   )
+  (label "-METER_RUN" (at 414.02 294.64 180)
+    (effects (font (size 1.27 1.27)) (justify right bottom))
+  )
   (label "+3V" (at 370.84 297.18 0)
     (effects (font (size 1.27 1.27)) (justify left bottom))
@@
     (effects (font (size 1.27 1.27)) (justify right bottom))
   )
+  (label "-METER_RUN" (at 33.02 246.38 180)
+    (effects (font (size 1.27 1.27)) (justify right bottom))
+  )
   (label "GND" (at 116.84 309.88 0)
     (effects (font (size 1.27 1.27)) (justify left bottom))
@@
     (effects (font (size 1.27 1.27)) (justify right bottom))
   )
+  (label "+RUN_PROG_LOAD_DOT_ON_RUN" (at 426.72 299.72 0)
+    (effects (font (size 1.27 1.27)) (justify left bottom))
+  )
   (label "GND" (at 243.84 233.68 0)
     (effects (font (size 1.27 1.27)) (justify left bottom))
@@
     (effects (font (size 1.27 1.27)) (justify right bottom))
   )
+  (label "+CPU_RUN" (at 45.72 307.34 0)
+    (effects (font (size 1.27 1.27)) (justify left bottom))
+  )
   (label "-U_BIT_13" (at 477.52 147.32 180)
     (effects (font (size 1.27 1.27)) (justify right bottom))
@@
     (effects (font (size 1.27 1.27)) (justify right bottom))
   )
+  (label "-RUN_LAMP_DR" (at 350.52 297.18 180)
+    (effects (font (size 1.27 1.27)) (justify right bottom))
+  )
   (label "+3V" (at 243.84 259.08 0)
     (effects (font (size 1.27 1.27)) (justify left bottom))
@@
     (effects (font (size 1.27 1.27)) (justify right bottom))
   )
+  (label "+CPU_RUN" (at 363.22 299.72 0)
+    (effects (font (size 1.27 1.27)) (justify left bottom))
+  )
   (label "+6V" (at 723.9 241.3 180)
     (effects (font (size 1.27 1.27)) (justify right bottom))
@@
     (effects (font (size 1.27 1.27)) (justify right bottom))
   )
+  (label "-RUN_LAMP_DR" (at 45.72 236.22 0)
+    (effects (font (size 1.27 1.27)) (justify left bottom))
+  )
   (label "GND" (at 497.84 271.78 0)
     (effects (font (size 1.27 1.27)) (justify left bottom))
@@
     (effects (font (size 1.27 1.27)) (justify left bottom))
   )
+  (label "-RUN_LAMP_DR" (at 223.52 233.68 180)
+    (effects (font (size 1.27 1.27)) (justify right bottom))
+  )
   (label "GND" (at 440.69 349.25 90)
     (effects (font (size 1.27 1.27)) (justify left bottom))
@@
     (effects (font (size 1.27 1.27)) (justify left bottom))
   )
+  (label "+48V" (at 311.15 58.42 180)
+    (effects (font (size 1.27 1.27)) (justify right bottom))
+  )
   (label "+3V" (at 688.34 106.68 0)
     (effects (font (size 1.27 1.27)) (justify left bottom))
@@
     (effects (font (size 1.27 1.27)) (justify left bottom))
   )
+  (label "-X6_PWR" (at 426.72 322.58 0)
+    (effects (font (size 1.27 1.27)) (justify left bottom))
+  )
   (label "+U_REG_8_PWR" (at 405.13 50.8 90)
     (effects (font (size 1.27 1.27)) (justify left bottom))
@@
     (effects (font (size 1.27 1.27)) (justify left bottom))
   )
+  (label "-CE_KEY_SW" (at 426.72 312.42 0)
+    (effects (font (size 1.27 1.27)) (justify left bottom))
+  )
   (label "+U_REG_15_PWR" (at 350.52 132.08 180)
     (effects (font (size 1.27 1.27)) (justify right bottom))
@@
     (effects (font (size 1.27 1.27)) (justify left bottom))
   )
+  (label "+48V" (at 210.82 226.06 180)
+    (effects (font (size 1.27 1.27)) (justify right bottom))
+  )
   (label "+3V" (at 751.84 297.18 0)
     (effects (font (size 1.27 1.27)) (justify left bottom))
@@
     (effects (font (size 1.27 1.27)) (justify left bottom))
   )
+  (label "+OSC_A_PWR" (at 426.72 302.26 0)
+    (effects (font (size 1.27 1.27)) (justify left bottom))
+  )
   (label "-U_BIT_0" (at 350.52 119.38 180)
     (effects (font (size 1.27 1.27)) (justify right bottom))
@@
     (effects (font (size 1.27 1.27)) (justify right bottom))
   )
+  (label "-ACCESS_DRIVE" (at 426.72 320.04 0)
+    (effects (font (size 1.27 1.27)) (justify left bottom))
+  )
   (label "+3V" (at 434.34 106.68 0)
     (effects (font (size 1.27 1.27)) (justify left bottom))
@@
     (effects (font (size 1.27 1.27)) (justify left bottom))
   )
+  (label "KW101_AN4" (at 414.02 299.72 180)
+    (effects (font (size 1.27 1.27)) (justify right bottom))
+  )
   (label "DU111_AF4" (at 350.52 162.56 180)
     (effects (font (size 1.27 1.27)) (justify right bottom))
@@
     (effects (font (size 1.27 1.27)) (justify left bottom))
   )
+  (label "KW101_AN4" (at 414.02 307.34 180)
+    (effects (font (size 1.27 1.27)) (justify right bottom))
+  )
   (label "GND" (at 815.34 271.78 0)
     (effects (font (size 1.27 1.27)) (justify left bottom))
@@
   )
   (label "GND" (at 402.59 43.18 90)
+    (effects (font (size 1.27 1.27)) (justify left bottom))
+  )
+  (label "KW101_AB4" (at 426.72 317.5 0)
     (effects (font (size 1.27 1.27)) (justify left bottom))
   )
@@
     (effects (font (size 1.27 1.27)) (justify left))
   )
+  (hierarchical_label "+48V" (shape input) (at 311.15 58.42 0)
+    (effects (font (size 1.27 1.27)) (justify left))
+  )
