File: 1130_backplane/01B-C1.kicad_sch (KiCad schematic)
At the start: 86 parts

Commit message: Finish page WZ051 and WZ061
Connections:
- net -SENSE_BIT_10: now reaches J509.a3 (Pin_a3)
- net -SENSE_BIT_10: now also J479.a2 (Pin_a2), J515.a3 (Pin_a3)
- net -SENSE_BIT_12: now reaches J509.a9 (Pin_a9)
- net -SENSE_BIT_12: now also J479.a4 (Pin_a4), J515.a9 (Pin_a9)
- net -SENSE_BIT_1: now reaches J433.a3 (Pin_a3)
- net -SENSE_BIT_1: now also J439.a3 (Pin_a3), J467.a3 (Pin_a3)
- net -SENSE_BIT_5: now reaches J433.a9 (Pin_a9)
- net -SENSE_BIT_5: now also J439.a9 (Pin_a9), J467.a8 (Pin_a8)
- net -SENSE_BIT_7: now reaches J438.a3 (Pin_a3)
- net -SENSE_BIT_7: now also J432.a3 (Pin_a3), J467.a10 (Pin_a10), J467.a7 (Pin_a7)
- net -SENSE_BIT_9: now reaches J438.a9 (Pin_a9)
- net -SENSE_BIT_9: now also J432.a9 (Pin_a9), J467.a12 (Pin_a12)
- net -SENSE_BIT_11: now reaches J513.a3 (Pin_a3)
- net -SENSE_BIT_11: now also J479.a3 (Pin_a3), J507.a3 (Pin_a3)
- net -SENSE_BIT_17: now reaches J513.a9 (Pin_a9)
- net -SENSE_BIT_17: now also J479.a10 (Pin_a10), J479.a7 (Pin_a7), J507.a9 (Pin_a9)
- net -SENSE_BIT_14: now reaches J510.a3 (Pin_a3)
- net -SENSE_BIT_14: now also J479.a6 (Pin_a6), J516.a3 (Pin_a3)
- net -SENSE_BIT_16: now reaches J510.a9 (Pin_a9)
- net -SENSE_BIT_16: now also J479.a9 (Pin_a9), J516.a9 (Pin_a9)
- net -SENSE_BIT_4: now reaches J441.a3 (Pin_a3)
- net -SENSE_BIT_4: now also J435.a3 (Pin_a3), J467.a6 (Pin_a6)
- net -SENSE_BIT_8: now reaches J441.a9 (Pin_a9)
- net -SENSE_BIT_8: now also J435.a9 (Pin_a9), J467.a11 (Pin_a11)
- net -SENSE_BIT_15: now reaches J508.a3 (Pin_a3)
- net -SENSE_BIT_15: now also J479.a8 (Pin_a8), J514.a3 (Pin_a3)
- net -SENSE_BIT_13: now reaches J508.a9 (Pin_a9)
- net -SENSE_BIT_13: now also J479.a1 (Pin_a1), J479.a5 (Pin_a5), J514.a9 (Pin_a9)
- net -SENSE_BIT_3: now reaches J434.a3 (Pin_a3)
- net -SENSE_BIT_3: now also J440.a3 (Pin_a3), J467.a1 (Pin_a1), J467.a5 (Pin_a5)
- net -SENSE_BIT_2: now reaches J434.a9 (Pin_a9)
- net -SENSE_BIT_2: now also J440.a9 (Pin_a9), J467.a4 (Pin_a4)
- net -SENSE_BIT_6: now reaches J442.a3 (Pin_a3)
- net -SENSE_BIT_6: now also J436.a3 (Pin_a3), J467.a9 (Pin_a9)
- net -SENSE_BIT_0: now reaches J442.a9 (Pin_a9)
- net -SENSE_BIT_0: now also J436.a9 (Pin_a9), J467.a2 (Pin_a2)
Other:
- note added: "5803475"
